Commit message: Robot Spawning in Gazebo

File: warehouse_robot_sim/urdf/omni_controller.urdf.xacro (robot description, xacro)
@@ -4,26 +4,12 @@
     <plugin name="object_controller" filename="libgazebo_ros_planar_move.so">
       <ros>
-<<<<<<< HEAD
-        <remapping>odom:=odom</remapping>
-      </ros>
-      <command_topic>cmd_vel</command_topic>
-      <odometry_topic>odom</odometry_topic>
-=======
         <remapping>odom:=odom/unfiltered</remapping>
       </ros>
       <command_topic>cmd_vel</command_topic>
       <odometry_topic>odom/unfiltered</odometry_topic>
->>>>>>> 2349e1b (Removed config error)
       <odometry_frame>odom</odometry_frame>
       <odometry_rate>20.0</odometry_rate>
       <robot_base_frame>base_footprint</robot_base_frame>
       <publish_odom>true</publish_odom>
-<<<<<<< HEAD
-      <publish_odom_tf>true</publish_odom_tf>
-    </plugin>
-  </gazebo>
-  </xacro:macro>
-</robot>
-=======
       <publish_odom_tf>false</publish_odom_tf>
     </plugin>
@@ -31,3 +17,2 @@
   </xacro:macro>
 </robot>
->>>>>>> 2349e1b (Removed config error)

Commit message: Robot spawning in gazebo

File: warehouse_robot_sim/urdf/omni_controller.urdf.xacro (robot description, xacro)
@@ -4,12 +4,20 @@
     <plugin name="object_controller" filename="libgazebo_ros_planar_move.so">
       <ros>
+<<<<<<< HEAD
         <remapping>odom:=odom</remapping>
       </ros>
       <command_topic>cmd_vel</command_topic>
       <odometry_topic>odom</odometry_topic>
+=======
+        <remapping>odom:=odom/unfiltered</remapping>
+      </ros>
+      <command_topic>cmd_vel</command_topic>
+      <odometry_topic>odom/unfiltered</odometry_topic>
+>>>>>>> 2349e1b (Removed config error)
       <odometry_frame>odom</odometry_frame>
       <odometry_rate>20.0</odometry_rate>
       <robot_base_frame>base_footprint</robot_base_frame>
       <publish_odom>true</publish_odom>
+<<<<<<< HEAD
       <publish_odom_tf>true</publish_odom_tf>
     </plugin>
@@ -17,2 +25,9 @@
   </xacro:macro>
 </robot>
+=======
+      <publish_odom_tf>false</publish_odom_tf>
+    </plugin>
+  </gazebo>
+  </xacro:macro>
+</robot>
+>>>>>>> 2349e1b (Removed config error)
