Commit message: Updated urdf

File: warehouse_robot_sim/urdf/TriBot_Oakd.urdf.xacro (robot description, xacro)
@@ -1,6 +1,14 @@
-<?xml version="1.0" encoding="utf-8"?>
-<robot name="TriOrb300P100">
- <!-- <xacro:include filename="$(find warehouse_robot_sim)/urdf/oakd.urdf.xacro" /> -->
-    <link name="TriOrb300P100_TopPlate">
+<?xml version="1.0" ?>
+<robot name="TriOrb300P100_Corrected">
+  <link name="base_link">
+    <inertial>
+      <origin xyz="0 0 0" rpy="0 0 0"/>
+      <mass value="1.0"/>
+      <inertia ixx="1.0" ixy="0.0" ixz="0.0" iyy="1.0" iyz="0.0" izz="1.0"/>
+    </inertial>
+    <visual/>
+    <collision/>
+  </link>
+  <link name="TriOrb300P100_TopPlate">
         <inertial>
             <origin xyz="1.5137191669958588e-13 -0.0002619661940188339 0.14268613534243857" rpy="0.0 -0.0 0.0" />
@@ -11,8 +19,8 @@
             <origin xyz="0.0 0.0 0.0" rpy="0.0 -0.0 0.0" />
             <geometry>
-                <mesh filename="../meshes/TriOrb300P100_TopPlate.stl" scale="0.001 0.001 0.001" />
+                <mesh filename="~/tribot/src/warehouse_robot_sim/meshes/TriOrb300P100_TopPlate.stl" scale="0.001 0.001 0.001" />
             </geometry>
             <material name="dark_gray">
-                <color rgba="0.01 0.01 0.01 2.0"/>
+                <color rgba="0.01 0.01 0.01 1.0"/>
             </material>
         </visual>
@@ -20,30 +28,14 @@
             <origin xyz="0.0 0.0 0.0" rpy="0.0 -0.0 0.0" />
             <geometry>
-                <mesh filename="../meshes/TriOrb300P100_TopPlate.stl" scale="0.001 0.001 0.001" />
-            </geometry>
-        </collision>
-    </link>
-    <!-- Add Camera Plugin -->
-    <gazebo>
-        <plugin name="oakd_camera" filename="liboakd_camera_plugin.so">
-            <topic_name>/oakd_camera</topic_name>
-            <frame_name>oakd_camera_frame</frame_name>
-            <camera_info_topic>/camera_info</camera_info_topic>
-        </plugin>
-    </gazebo>
-    <!-- Add 3-Wheel Omni-Drive Plugin -->
-    <gazebo>
-        <plugin name="omni_drive_plugin" filename="libgazebo_omni_drive_plugin.so">
-            <robot_base_frame>base_link</robot_base_frame>
-            <wheel_radius>0.05</wheel_radius>
-            <wheel_separation>0.3</wheel_separation>
-            <wheel_joints>
-                <joint>left_wheel_joint</joint>
-                <joint>right_wheel_joint</joint>
-                <joint>back_wheel_joint</joint>
-            </wheel_joints>
-        </plugin>
-    </gazebo>
-    <link name="TriOrb300P100_Ball100_1">
+                <mesh filename="~/tribot/src/warehouse_robot_sim/meshes/TriOrb300P100_TopPlate.stl" scale="0.001 0.001 0.001" />
+            </geometry>
+        </collision>
+  </link>
+  <joint name="TriOrb300P100_TopPlate_joint" type="fixed">
+    <parent link="base_link"/>
+    <child link="TriOrb300P100_TopPlate"/>
+    <origin xyz="0 0 0" rpy="0 0 0"/>
+  </joint>
+  <link name="TriOrb300P100_Ball100_1">
         <visual>
             <geometry>
@@ -52,5 +44,5 @@
             <origin xyz="0 0.187 0.05" rpy="0 0 0"/>
             <material name="triorb_blue">
-                <color rgba="0.1333333333333333 0.2313725490196078 0.5019607843137255 2.0"/>
+                <color rgba="0.1333333333333333 0.2313725490196078 0.5019607843137255 1.0"/>
             </material>
         </visual>
@@ -61,6 +53,11 @@
             <origin xyz="0 0.187 0.05" rpy="0 0 0"/>
         </collision>
-    </link>
-    <link name="TriOrb300P100_Ball100_2">
+  </link>
+  <joint name="TriOrb300P100_Ball100_1_joint" type="fixed">
+    <parent link="base_link"/>
+    <child link="TriOrb300P100_Ball100_1"/>
+    <origin xyz="0 0 0" rpy="0 0 0"/>
+  </joint>
+  <link name="TriOrb300P100_Ball100_2">
         <visual>
             <geometry>
@@ -69,5 +66,5 @@
             <origin xyz="0.162 -0.094 0.05" rpy="0 0 0"/>
             <material name="triorb_blue">
-                <color rgba="0.1333333333333333 0.2313725490196078 0.5019607843137255 2.0"/>
+                <color rgba="0.1333333333333333 0.2313725490196078 0.5019607843137255 1.0"/>
             </material>
         </visual>
@@ -78,6 +75,6 @@
             <origin xyz="0.162 -0.094 0.05" rpy="0 0 0"/>
         </collision>
-    </link>
-    <link name="TriOrb300P100_Ball100_3">
+  </link>
+  <link name="TriOrb300P100_Ball100_3">
         <visual>
             <geometry>
@@ -86,5 +83,5 @@
             <origin xyz="-0.162 -0.094 0.05" rpy="0 0 0"/>
             <material name="triorb_blue">
-                <color rgba="0.1333333333333333 0.2313725490196078 0.5019607843137255 2.0"/>
+                <color rgba="0.1333333333333333 0.2313725490196078 0.5019607843137255 1.0"/>
             </material>
         </visual>
@@ -95,6 +92,16 @@
             <origin xyz="-0.162 -0.094 0.05" rpy="0 0 0"/>
         </collision>
-    </link>
-    <link name="TriOrb300P100_PlateA_PlateA-1">
+  </link>
+  <joint name="TriOrb300P100_Ball100_2_joint" type="fixed">
+    <parent link="base_link"/>
+    <child link="TriOrb300P100_Ball100_2"/>
+    <origin xyz="0 0 0" rpy="0 0 0"/>
+  </joint>
+  <joint name="TriOrb300P100_Ball100_3_joint" type="fixed">
+    <parent link="base_link"/>
+    <child link="TriOrb300P100_Ball100_3"/>
+    <origin xyz="0 0 0" rpy="0 0 0"/>
+  </joint>
+  <link name="TriOrb300P100_PlateA_PlateA-1">
         <inertial>
             <mass value="0.39569212966450507" />
@@ -103,8 +110,8 @@
             <origin xyz="0.0 -0.131 0.064" rpy="1.5708 0.0 0.0" />
             <geometry>
-                <mesh filename="../meshes/TriOrb300P100_PlateA_PlateA-1.stl" scale="0.001 0.001 0.001" />
+                <mesh filename="~/tribot/src/warehouse_robot_sim/meshes/TriOrb300P100_PlateA_PlateA-1.stl" scale="0.001 0.001 0.001" />
             </geometry>
             <material name="aluminum">
-                <color rgba="0.5 0.5490196078431373 0.5333333333333333 2.0"/>
+                <color rgba="0.5 0.5490196078431373 0.5333333333333333 1.0"/>
             </material>
         </visual>
@@ -115,6 +122,11 @@
             </geometry>
         </collision>
-    </link>
-    <link name="TriOrb300P100_PlateA_PlateA-2">
+  </link>
+  <joint name="TriOrb300P100_PlateA_PlateA-1_joint" type="fixed">
+    <parent link="base_link"/>
+    <child link="TriOrb300P100_PlateA_PlateA-1"/>
+    <origin xyz="0 0 0" rpy="0 0 0"/>
+  </joint>
+  <link name="TriOrb300P100_PlateA_PlateA-2">
         <inertial>
             <mass value="0.39569212966450507" />
@@ -123,8 +135,8 @@
             <origin xyz="0.115 0.067 0.064" rpy="1.5708 0.0 2.0944" />
             <geometry>
-                <mesh filename="../meshes/TriOrb300P100_PlateA_PlateA-1.stl" scale="0.001 0.001 0.001" />
+                <mesh filename="~/tribot/src/warehouse_robot_sim/meshes/TriOrb300P100_PlateA_PlateA-1.stl" scale="0.001 0.001 0.001" />
             </geometry>
             <material name="aluminum">
-                <color rgba="0.5 0.5490196078431373 0.5333333333333333 2.0"/>
+                <color rgba="0.5 0.5490196078431373 0.5333333333333333 1.0"/>
             </material>
         </visual>
@@ -132,9 +144,9 @@
             <origin xyz="0.115 0.067 0.064" rpy="1.5708 0.0 2.0944" />
             <geometry>
-                <mesh filename="../meshes/TriOrb300P100_PlateA_PlateA-1.stl" scale="0.001 0.001 0.001" />
-            </geometry>
-        </collision>
-    </link>
-    <link name="TriOrb300P100_PlateA_PlateA-3">
+                <mesh filename="~/tribot/src/warehouse_robot_sim/meshes/TriOrb300P100_PlateA_PlateA-1.stl" scale="0.001 0.001 0.001" />
+            </geometry>
+        </collision>
+  </link>
+  <link name="TriOrb300P100_PlateA_PlateA-3">
         <inertial>
             <mass value="0.39569212966450507" />
@@ -143,8 +155,8 @@
             <origin xyz="-0.115 0.067 0.064" rpy="1.5708 0.0 -2.0944" />
             <geometry>
-                <mesh filename="../meshes/TriOrb300P100_PlateA_PlateA-1.stl" scale="0.001 0.001 0.001" />
+                <mesh filename="~/tribot/src/warehouse_robot_sim/meshes/TriOrb300P100_PlateA_PlateA-1.stl" scale="0.001 0.001 0.001" />
             </geometry>
             <material name="aluminum">
-                <color rgba="0.5 0.5490196078431373 0.5333333333333333 2.0"/>
+                <color rgba="0.5 0.5490196078431373 0.5333333333333333 1.0"/>
             </material>
         </visual>
@@ -152,9 +164,19 @@
             <origin xyz="-0.115 0.067 0.064" rpy="1.5708 0.0 -2.0944" />
             <geometry>
-                <mesh filename="../meshes/TriOrb300P100_PlateA_PlateA-1.stl" scale="0.001 0.001 0.001" />
-            </geometry>
-        </collision>
-    </link>
-    <link name="TriOrb300P100_Casters_BlockC_BlockC1">
+                <mesh filename="~/tribot/src/warehouse_robot_sim/meshes/TriOrb300P100_PlateA_PlateA-1.stl" scale="0.001 0.001 0.001" />
+            </geometry>
+        </collision>
+  </link>
+  <joint name="TriOrb300P100_PlateA_PlateA-2_joint" type="fixed">
+    <parent link="base_link"/>
+    <child link="TriOrb300P100_PlateA_PlateA-2"/>
+    <origin xyz="0 0 0" rpy="0 0 0"/>
+  </joint>
+  <joint name="TriOrb300P100_PlateA_PlateA-3_joint" type="fixed">
+    <parent link="base_link"/>
+    <child link="TriOrb300P100_PlateA_PlateA-3"/>
+    <origin xyz="0 0 0" rpy="0 0 0"/>
+  </joint>
+  <link name="TriOrb300P100_Casters_BlockC_BlockC1">
         <inertial>
             <origin xyz="0.010662803863432657 -2.8483899861735884e-17 0.017741942156625452" rpy="0.0 0.0 0.0" />
@@ -165,8 +187,8 @@
             <origin xyz="0.0 0.226 0.138" rpy="0.0 3.1415 -1.5708" />
             <geometry>
-                <mesh filename="../meshes/TriOrb300P100_Casters_BlockC_BlockC1.stl" scale="0.001 0.001 0.001" />
+                <mesh filename="~/tribot/src/warehouse_robot_sim/meshes/TriOrb300P100_Casters_BlockC_BlockC1.stl" scale="0.001 0.001 0.001" />
             </geometry>
             <material name="dark_gray">
-                <color rgba="0.01 0.01 0.01 2.0"/>
+                <color rgba="0.01 0.01 0.01 1.0"/>
             </material>
         </visual>
@@ -174,9 +196,9 @@
             <origin xyz="0.0 0.226 0.138" rpy="0.0 3.1415 -1.5708" />
             <geometry>
-                <mesh filename="../meshes/TriOrb300P100_Casters_BlockC_BlockC1.stl" scale="0.001 0.001 0.001" />
-            </geometry>
-        </collision>
-    </link>
-    <link name="TriOrb300P100_Casters_BlockC_BlockC2">
+                <mesh filename="~/tribot/src/warehouse_robot_sim/meshes/TriOrb300P100_Casters_BlockC_BlockC1.stl" scale="0.001 0.001 0.001" />
+            </geometry>
+        </collision>
+  </link>
+  <link name="TriOrb300P100_Casters_BlockC_BlockC2">
         <inertial>
             <origin xyz="0.010662803863432657 -2.8483899861735884e-17 0.017741942156625452" rpy="0.0 0.0 0.0" />
@@ -187,8 +209,8 @@
             <origin xyz="-0.196 -0.113 0.138" rpy="0.0 3.1415 0.521" />
             <geometry>
-                <mesh filename="../meshes/TriOrb300P100_Casters_BlockC_BlockC1.stl" scale="0.001 0.001 0.001" />
+                <mesh filename="~/tribot/src/warehouse_robot_sim/meshes/TriOrb300P100_Casters_BlockC_BlockC1.stl" scale="0.001 0.001 0.001" />
             </geometry>
             <material name="dark_gray">
-                <color rgba="0.01 0.01 0.01 2.0"/>
+                <color rgba="0.01 0.01 0.01 1.0"/>
             </material>
         </visual>
@@ -196,9 +218,9 @@
             <origin xyz="-0.196 -0.113 0.138" rpy="0.0 3.1415 0.521" />
             <geometry>
-                <mesh filename="../meshes/TriOrb300P100_Casters_BlockC_BlockC1.stl" scale="0.001 0.001 0.001" />
-            </geometry>
-        </collision>
-    </link>
-    <link name="TriOrb300P100_Casters_BlockC_BlockC3">
+                <mesh filename="~/tribot/src/warehouse_robot_sim/meshes/TriOrb300P100_Casters_BlockC_BlockC1.stl" scale="0.001 0.001 0.001" />
+            </geometry>
+        </collision>
+  </link>
+  <link name="TriOrb300P100_Casters_BlockC_BlockC3">
         <inertial>
             <origin xyz="0.010662803863432657 -2.8483899861735884e-17 0.017741942156625452" rpy="0.0 0.0 0.0" />
@@ -209,8 +231,8 @@
             <origin xyz="0.196 -0.113 0.138" rpy="0.0 3.1415 2.6154" />
             <geometry>
-                <mesh filename="../meshes/TriOrb300P100_Casters_BlockC_BlockC1.stl" scale="0.001 0.001 0.001" />
+                <mesh filename="~/tribot/src/warehouse_robot_sim/meshes/TriOrb300P100_Casters_BlockC_BlockC1.stl" scale="0.001 0.001 0.001" />
             </geometry>
             <material name="dark_gray">
-                <color rgba="0.01 0.01 0.01 2.0"/>
+                <color rgba="0.01 0.01 0.01 1.0"/>
             </material>
         </visual>
@@ -218,9 +240,24 @@
             <origin xyz="0.196 -0.113 0.138" rpy="0.0 3.1415 2.6154" />
             <geometry>
-                <mesh filename="../meshes/TriOrb300P100_Casters_BlockC_BlockC1.stl" scale="0.001 0.001 0.001" />
-            </geometry>
-        </collision>
-    </link>
-    <link name="TriOrb300P100_Casters_BlockC_Pall1a">
+                <mesh filename="~/tribot/src/warehouse_robot_sim/meshes/TriOrb300P100_Casters_BlockC_BlockC1.stl" scale="0.001 0.001 0.001" />
+            </geometry>
+        </collision>
+  </link>
+  <joint name="TriOrb300P100_Casters_BlockC_BlockC1_joint" type="fixed">
+    <parent link="base_link"/>
+    <child link="TriOrb300P100_Casters_BlockC_BlockC1"/>
+    <origin xyz="0 0 0" rpy="0 0 0"/>
+  </joint>
+  <joint name="TriOrb300P100_Casters_BlockC_BlockC2_joint" type="fixed">
+    <parent link="base_link"/>
+    <child link="TriOrb300P100_Casters_BlockC_BlockC2"/>
+    <origin xyz="0 0 0" rpy="0 0 0"/>
+  </joint>
+  <joint name="TriOrb300P100_Casters_BlockC_BlockC3_joint" type="fixed">
+    <parent link="base_link"/>
+    <child link="TriOrb300P100_Casters_BlockC_BlockC3"/>
+    <origin xyz="0 0 0" rpy="0 0 0"/>
+  </joint>
+  <link name="TriOrb300P100_Casters_BlockC_Pall1a">
         <inertial>
             <origin xyz="-0.0009138193356166049 0.00010427567796962438 0.05387638922345278" rpy="0.0 0.0 0.0" />
@@ -231,8 +268,8 @@
             <origin xyz="-0.057 0.222 0.138" rpy="0 3.1415 2.617901" />
             <geometry>
-                <mesh filename="../meshes/TriOrb300P100_Casters_BlockC_Pall.stl" scale="0.001 0.001 0.001" />
+                <mesh filename="~/tribot/src/warehouse_robot_sim/meshes/TriOrb300P100_Casters_BlockC_Pall.stl" scale="0.001 0.001 0.001" />
             </geometry>
             <material name="dark_gray">
-                <color rgba="0.01 0.01 0.01 2.0"/>
+                <color rgba="0.01 0.01 0.01 1.0"/>
             </material>
         </visual>
@@ -240,9 +277,9 @@
             <origin xyz="-0.057 0.222 0.138" rpy="0 3.1415 2.617901" />
             <geometry>
-                <mesh filename="../meshes/TriOrb300P100_Casters_BlockC_Pall.stl" scale="0.001 0.001 0.001" />
-            </geometry>
-        </collision>
-    </link>
-    <link name="TriOrb300P100_Casters_BlockC_Pall1b">
+                <mesh filename="~/tribot/src/warehouse_robot_sim/meshes/TriOrb300P100_Casters_BlockC_Pall.stl" scale="0.001 0.001 0.001" />
+            </geometry>
+        </collision>
+  </link>
+  <link name="TriOrb300P100_Casters_BlockC_Pall1b">
         <inertial>
             <origin xyz="-0.0009138193356166049 0.00010427567796962438 0.05387638922345278" rpy="0.0 0.0 0.0" />
@@ -253,8 +290,8 @@
             <origin xyz="0.057 0.222 0.138" rpy="0 3.1415 0.523599" />
             <geometry>
-                <mesh filename="../meshes/TriOrb300P100_Casters_BlockC_Pall.stl" scale="0.001 0.001 0.001" />
+                <mesh filename="~/tribot/src/warehouse_robot_sim/meshes/TriOrb300P100_Casters_BlockC_Pall.stl" scale="0.001 0.001 0.001" />
             </geometry>
             <material name="dark_gray">
-                <color rgba="0.01 0.01 0.01 2.0"/>
+                <color rgba="0.01 0.01 0.01 1.0"/>
             </material>
         </visual>
@@ -262,9 +299,9 @@
             <origin xyz="0.057 0.222 0.138" rpy="0 3.1415 0.523599" />
             <geometry>
-                <mesh filename="../meshes/TriOrb300P100_Casters_BlockC_Pall.stl" scale="0.001 0.001 0.001" />
-            </geometry>
-        </collision>
-    </link>
-    <link name="TriOrb300P100_Casters_BlockC_Pall2a">
+                <mesh filename="~/tribot/src/warehouse_robot_sim/meshes/TriOrb300P100_Casters_BlockC_Pall.stl" scale="0.001 0.001 0.001" />
+            </geometry>
+        </collision>
+  </link>
+  <link name="TriOrb300P100_Casters_BlockC_Pall2a">
         <inertial>
             <origin xyz="-0.0009138193356166049 0.00010427567796962438 0.05387638922345278" rpy="0.0 0.0 0.0" />
@@ -275,8 +312,8 @@
             <origin xyz="0.221 -0.062 0.138" rpy="0 3.1415 0.521" />
             <geometry>
-                <mesh filename="../meshes/TriOrb300P100_Casters_BlockC_Pall.stl" scale="0.001 0.001 0.001" />
+                <mesh filename="~/tribot/src/warehouse_robot_sim/meshes/TriOrb300P100_Casters_BlockC_Pall.stl" scale="0.001 0.001 0.001" />
             </geometry>
             <material name="dark_gray">
-                <color rgba="0.01 0.01 0.01 2.0"/>
+                <color rgba="0.01 0.01 0.01 1.0"/>
             </material>
         </visual>
@@ -284,9 +321,9 @@
             <origin xyz="0.221 -0.062 0.138" rpy="0 3.1415 0.521" />
             <geometry>
-                <mesh filename="../meshes/TriOrb300P100_Casters_BlockC_Pall.stl" scale="0.001 0.001 0.001" />
-            </geometry>
-        </collision>
-    </link>
-    <link name="TriOrb300P100_Casters_BlockC_Pall2b">
+                <mesh filename="~/tribot/src/warehouse_robot_sim/meshes/TriOrb300P100_Casters_BlockC_Pall.stl" scale="0.001 0.001 0.001" />
+            </geometry>
+        </collision>
+  </link>
+  <link name="TriOrb300P100_Casters_BlockC_Pall2b">
         <inertial>
             <origin xyz="-0.0009138193356166049 0.00010427567796962438 0.05387638922345278" rpy="0.0 0.0 0.0" />
@@ -297,8 +334,8 @@
             <origin xyz="0.164 -0.16 0.138" rpy="0 3.1415 -1.5734" />
             <geometry>
-                <mesh filename="../meshes/TriOrb300P100_Casters_BlockC_Pall.stl" scale="0.001 0.001 0.001" />
+                <mesh filename="~/tribot/src/warehouse_robot_sim/meshes/TriOrb300P100_Casters_BlockC_Pall.stl" scale="0.001 0.001 0.001" />
             </geometry>
             <material name="dark_gray">
-                <color rgba="0.01 0.01 0.01 2.0"/>
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