Commit message: Updated Robot without camera

File: warehouse_robot_sim/urdf/TriBot_Oakd.urdf.xacro (robot description, xacro)
@@ -7,28 +7,41 @@
       <inertia ixx="1.0" ixy="0.0" ixz="0.0" iyy="1.0" iyz="0.0" izz="1.0"/>
     </inertial>
-    <visual/>
-    <collision/>
+    <visual name="TriOrb300P100_UnderPlate_visual">
+        <origin xyz="0.0 0.0 0.0" rpy="0.0 0.0 0.0" />
+        <geometry>
+            <mesh filename="~/tribot/src/warehouse_robot_sim/meshes/TriOrb300P100_UnderPlate.stl" scale="0.001 0.001 0.001" />
+        </geometry>
+        <material name="sus">
+            <color rgba="0.753 0.753 0.753 1.0"/>
+        </material>
+    </visual>
+    <collision name="TriOrb300P100_UnderPlate_collision">
+        <origin xyz="0.0 0.0 0.0" rpy="0.0 0.0 0.0" />
+        <geometry>
+            <mesh filename="~/tribot/src/warehouse_robot_sim/meshes/TriOrb300P100_UnderPlate.stl" scale="0.001 0.001 0.001" />
+        </geometry>
+    </collision>
   </link>
   <link name="TriOrb300P100_TopPlate">
-        <inertial>
-            <origin xyz="1.5137191669958588e-13 -0.0002619661940188339 0.14268613534243857" rpy="0.0 -0.0 0.0" />
-            <mass value="8.182272397574748" />
-            <inertia ixx="0.13232877336076157" iyy="0.13289875477595392" izz="0.2650914872635593" ixy="4.4043453928310243e-14" iyz="5.610845970076186e-08" ixz="7.989679922409314e-17" />
-        </inertial>
-        <visual name="TriOrb300P100_TopPlate_visual">
-            <origin xyz="0.0 0.0 0.0" rpy="0.0 -0.0 0.0" />
-            <geometry>
-                <mesh filename="~/tribot/src/warehouse_robot_sim/meshes/TriOrb300P100_TopPlate.stl" scale="0.001 0.001 0.001" />
-            </geometry>
-            <material name="dark_gray">
-                <color rgba="0.01 0.01 0.01 1.0"/>
-            </material>
-        </visual>
-        <collision name="TriOrb300P100_TopPlate_collision">
-            <origin xyz="0.0 0.0 0.0" rpy="0.0 -0.0 0.0" />
-            <geometry>
-                <mesh filename="~/tribot/src/warehouse_robot_sim/meshes/TriOrb300P100_TopPlate.stl" scale="0.001 0.001 0.001" />
-            </geometry>
-        </collision>
+    <inertial>
+        <origin xyz="1.5137191669958588e-13 -0.0002619661940188339 0.14268613534243857" rpy="0.0 -0.0 0.0" />
+        <mass value="8.182272397574748" />
+        <inertia ixx="0.13232877336076157" iyy="0.13289875477595392" izz="0.2650914872635593" ixy="4.4043453928310243e-14" iyz="5.610845970076186e-08" ixz="7.989679922409314e-17" />
+    </inertial>
+    <visual name="TriOrb300P100_TopPlate_visual">
+        <origin xyz="0.0 0.0 0.0" rpy="0.0 -0.0 0.0" />
+        <geometry>
+            <mesh filename="~/tribot/src/warehouse_robot_sim/meshes/TriOrb300P100_TopPlate.stl" scale="0.001 0.001 0.001" />
+        </geometry>
+        <material name="dark_gray">
+            <color rgba="0.01 0.01 0.01 1.0"/>
+        </material>
+    </visual>
+    <collision name="TriOrb300P100_TopPlate_collision">
+        <origin xyz="0.0 0.0 0.0" rpy="0.0 -0.0 0.0" />
+        <geometry>
+            <mesh filename="~/tribot/src/warehouse_robot_sim/meshes/TriOrb300P100_TopPlate.stl" scale="0.001 0.001 0.001" />
+        </geometry>
+    </collision>
   </link>
   <joint name="TriOrb300P100_TopPlate_joint" type="fixed">
@@ -38,19 +51,24 @@
   </joint>
   <link name="TriOrb300P100_Ball100_1">
-        <visual>
-            <geometry>
-                <sphere radius="0.05"/>
-            </geometry>
-            <origin xyz="0 0.187 0.05" rpy="0 0 0"/>
-            <material name="triorb_blue">
-                <color rgba="0.1333333333333333 0.2313725490196078 0.5019607843137255 1.0"/>
-            </material>
-        </visual>
-        <collision>
-            <geometry>
-                <sphere radius="0.05"/>
-            </geometry>
-            <origin xyz="0 0.187 0.05" rpy="0 0 0"/>
-        </collision>
+    <inertial>
+        <origin xyz="0 0 0" rpy="0 0 0" />
+        <mass value="0.01" />
+        <inertia ixx="0.0001" ixy="0.0" ixz="0.0" iyy="0.0001" iyz="0.0" izz="0.0001" />
+    </inertial>
+    <visual>
+        <geometry>
+            <sphere radius="0.05"/>
+        </geometry>
+        <origin xyz="0 0.187 0.05" rpy="0 0 0"/>
+        <material name="triorb_blue">
+            <color rgba="0.1333333333333333 0.2313725490196078 0.5019607843137255 1.0"/>
+        </material>
+    </visual>
+    <collision>
+        <geometry>
+            <sphere radius="0.05"/>
+        </geometry>
+        <origin xyz="0 0.187 0.05" rpy="0 0 0"/>
+    </collision>
   </link>
   <joint name="TriOrb300P100_Ball100_1_joint" type="fixed">
@@ -60,36 +78,46 @@
   </joint>
   <link name="TriOrb300P100_Ball100_2">
-        <visual>
-            <geometry>
-                <sphere radius="0.05"/>
-            </geometry>
-            <origin xyz="0.162 -0.094 0.05" rpy="0 0 0"/>
-            <material name="triorb_blue">
-                <color rgba="0.1333333333333333 0.2313725490196078 0.5019607843137255 1.0"/>
-            </material>
-        </visual>
-        <collision>
-            <geometry>
-                <sphere radius="0.05"/>
-            </geometry>
-            <origin xyz="0.162 -0.094 0.05" rpy="0 0 0"/>
-        </collision>
+    <inertial>
+        <origin xyz="0 0 0" rpy="0 0 0" />
+        <mass value="0.01" />
+        <inertia ixx="0.0001" ixy="0.0" ixz="0.0" iyy="0.0001" iyz="0.0" izz="0.0001" />
+    </inertial>
+    <visual>
+        <geometry>
+            <sphere radius="0.05"/>
+        </geometry>
+        <origin xyz="0.162 -0.094 0.05" rpy="0 0 0"/>
+        <material name="triorb_blue">
+            <color rgba="0.1333333333333333 0.2313725490196078 0.5019607843137255 1.0"/>
+        </material>
+    </visual>
+    <collision>
+        <geometry>
+            <sphere radius="0.05"/>
+        </geometry>
+        <origin xyz="0.162 -0.094 0.05" rpy="0 0 0"/>
+    </collision>
   </link>
   <link name="TriOrb300P100_Ball100_3">
-        <visual>
-            <geometry>
-                <sphere radius="0.05"/>
-            </geometry>
-            <origin xyz="-0.162 -0.094 0.05" rpy="0 0 0"/>
-            <material name="triorb_blue">
-                <color rgba="0.1333333333333333 0.2313725490196078 0.5019607843137255 1.0"/>
-            </material>
-        </visual>
-        <collision>
-            <geometry>
-                <sphere radius="0.05"/>
-            </geometry>
-            <origin xyz="-0.162 -0.094 0.05" rpy="0 0 0"/>
-        </collision>
+    <inertial>
+        <origin xyz="0 0 0" rpy="0 0 0" />
+        <mass value="0.01" />
+        <inertia ixx="0.0001" ixy="0.0" ixz="0.0" iyy="0.0001" iyz="0.0" izz="0.0001" />
+    </inertial>
+    <visual>
+        <geometry>
+            <sphere radius="0.05"/>
+        </geometry>
+        <origin xyz="-0.162 -0.094 0.05" rpy="0 0 0"/>
+        <material name="triorb_blue">
+            <color rgba="0.1333333333333333 0.2313725490196078 0.5019607843137255 1.0"/>
+        </material>
+    </visual>
+    <collision>
+        <geometry>
+            <sphere radius="0.05"/>
+        </geometry>
+        <origin xyz="-0.162 -0.094 0.05" rpy="0 0 0"/>
+    </collision>
   </link>
   <joint name="TriOrb300P100_Ball100_2_joint" type="fixed">
@@ -104,22 +132,23 @@
   </joint>
   <link name="TriOrb300P100_PlateA_PlateA-1">
-        <inertial>
-            <mass value="0.39569212966450507" />
-        </inertial>
-        <visual name="TriOrb300P100_PlateA_PlateA-1_visual">
-            <origin xyz="0.0 -0.131 0.064" rpy="1.5708 0.0 0.0" />
-            <geometry>
-                <mesh filename="~/tribot/src/warehouse_robot_sim/meshes/TriOrb300P100_PlateA_PlateA-1.stl" scale="0.001 0.001 0.001" />
-            </geometry>
-            <material name="aluminum">
-                <color rgba="0.5 0.5490196078431373 0.5333333333333333 1.0"/>
-            </material>
-        </visual>
-        <collision name="TriOrb300P100_PlateA_PlateA-1_collision">
-            <origin xyz="0.0 -0.131 0.064" rpy="1.5708 0.0 0.0" />
-            <geometry>
-                <mesh filename="../meshes/TriOrb300P100_PlateA_PlateA-1.stl" scale="0.001 0.001 0.001" />
-            </geometry>
-        </collision>
+    <inertial>
+        <mass value="0.39569212966450507" />
+        <inertia ixx="0.0001" ixy="0.0" ixz="0.0" iyy="0.0001" iyz="0.0" izz="0.0001" />
+    </inertial>
+    <visual name="TriOrb300P100_PlateA_PlateA-1_visual">
+        <origin xyz="0.0 -0.131 0.064" rpy="1.5708 0.0 0.0" />
+        <geometry>
+            <mesh filename="~/tribot/src/warehouse_robot_sim/meshes/TriOrb300P100_PlateA_PlateA-1.stl" scale="0.001 0.001 0.001" />
+        </geometry>
+        <material name="aluminum">
+            <color rgba="0.5 0.5490196078431373 0.5333333333333333 1.0"/>
+        </material>
+    </visual>
+    <collision name="TriOrb300P100_PlateA_PlateA-1_collision">
+        <origin xyz="0.0 -0.131 0.064" rpy="1.5708 0.0 0.0" />
+        <geometry>
+            <mesh filename="../meshes/TriOrb300P100_PlateA_PlateA-1.stl" scale="0.001 0.001 0.001" />
+        </geometry>
+    </collision>
   </link>
   <joint name="TriOrb300P100_PlateA_PlateA-1_joint" type="fixed">
@@ -129,42 +158,44 @@
   </joint>
   <link name="TriOrb300P100_PlateA_PlateA-2">
-        <inertial>
-            <mass value="0.39569212966450507" />
-        </inertial>
-        <visual name="TriOrb300P100_PlateA_PlateA-2_visual">
-            <origin xyz="0.115 0.067 0.064" rpy="1.5708 0.0 2.0944" />
-            <geometry>
-                <mesh filename="~/tribot/src/warehouse_robot_sim/meshes/TriOrb300P100_PlateA_PlateA-1.stl" scale="0.001 0.001 0.001" />
-            </geometry>
-            <material name="aluminum">
-                <color rgba="0.5 0.5490196078431373 0.5333333333333333 1.0"/>
-            </material>
-        </visual>
-        <collision name="TriOrb300P100_PlateA_PlateA-2_collision">
-            <origin xyz="0.115 0.067 0.064" rpy="1.5708 0.0 2.0944" />
-            <geometry>
-                <mesh filename="~/tribot/src/warehouse_robot_sim/meshes/TriOrb300P100_PlateA_PlateA-1.stl" scale="0.001 0.001 0.001" />
-            </geometry>
-        </collision>
+    <inertial>
+        <mass value="0.39569212966450507" />
+        <inertia ixx="0.0001" ixy="0.0" ixz="0.0" iyy="0.0001" iyz="0.0" izz="0.0001" />
+    </inertial>
+    <visual name="TriOrb300P100_PlateA_PlateA-2_visual">
+        <origin xyz="0.115 0.067 0.064" rpy="1.5708 0.0 2.0944" />
+        <geometry>
+            <mesh filename="~/tribot/src/warehouse_robot_sim/meshes/TriOrb300P100_PlateA_PlateA-1.stl" scale="0.001 0.001 0.001" />
+        </geometry>
+        <material name="aluminum">
+            <color rgba="0.5 0.5490196078431373 0.5333333333333333 1.0"/>
+        </material>
+    </visual>
+    <collision name="TriOrb300P100_PlateA_PlateA-2_collision">
+        <origin xyz="0.115 0.067 0.064" rpy="1.5708 0.0 2.0944" />
+        <geometry>
+            <mesh filename="~/tribot/src/warehouse_robot_sim/meshes/TriOrb300P100_PlateA_PlateA-1.stl" scale="0.001 0.001 0.001" />
+        </geometry>
+    </collision>
   </link>
   <link name="TriOrb300P100_PlateA_PlateA-3">
-        <inertial>
-            <mass value="0.39569212966450507" />
-        </inertial>
-        <visual name="TriOrb300P100_PlateA_PlateA-3_visual">
-            <origin xyz="-0.115 0.067 0.064" rpy="1.5708 0.0 -2.0944" />
-            <geometry>
-                <mesh filename="~/tribot/src/warehouse_robot_sim/meshes/TriOrb300P100_PlateA_PlateA-1.stl" scale="0.001 0.001 0.001" />
-            </geometry>
-            <material name="aluminum">
-                <color rgba="0.5 0.5490196078431373 0.5333333333333333 1.0"/>
-            </material>
-        </visual>
-        <collision name="TriOrb300P100_PlateA_PlateA-3_collision">
-            <origin xyz="-0.115 0.067 0.064" rpy="1.5708 0.0 -2.0944" />
-            <geometry>
-                <mesh filename="~/tribot/src/warehouse_robot_sim/meshes/TriOrb300P100_PlateA_PlateA-1.stl" scale="0.001 0.001 0.001" />
-            </geometry>
-        </collision>
+    <inertial>
+        <mass value="0.39569212966450507" />
+        <inertia ixx="0.0001" ixy="0.0" ixz="0.0" iyy="0.0001" iyz="0.0" izz="0.0001" />
+    </inertial>
+    <visual name="TriOrb300P100_PlateA_PlateA-3_visual">
+        <origin xyz="-0.115 0.067 0.064" rpy="1.5708 0.0 -2.0944" />
+        <geometry>
+            <mesh filename="~/tribot/src/warehouse_robot_sim/meshes/TriOrb300P100_PlateA_PlateA-1.stl" scale="0.001 0.001 0.001" />
+        </geometry>
+        <material name="aluminum">
+            <color rgba="0.5 0.5490196078431373 0.5333333333333333 1.0"/>
+        </material>
+    </visual>
+    <collision name="TriOrb300P100_PlateA_PlateA-3_collision">
+        <origin xyz="-0.115 0.067 0.064" rpy="1.5708 0.0 -2.0944" />
+        <geometry>
+            <mesh filename="~/tribot/src/warehouse_robot_sim/meshes/TriOrb300P100_PlateA_PlateA-1.stl" scale="0.001 0.001 0.001" />
+        </geometry>
+    </collision>
   </link>
   <joint name="TriOrb300P100_PlateA_PlateA-2_joint" type="fixed">

Commit message: urdf without oakd

File: warehouse_robot_sim/urdf/TriBot_Oakd.urdf.xacro (robot description, xacro)
@@ -1,4 +1,4 @@
 <?xml version="1.0" ?>
-<robot name="TriOrb300P100_Corrected">
+<robot name="TriOrb300P100">
   <link name="base_link">
     <inertial>
@@ -23,4 +23,116 @@
     </collision>
   </link>
+     <!-- Wheel 1 Definition -->
+   <link name="wheel1">
+       <inertial>
+           <mass value="1.0"/> <!-- Adjust mass as needed -->
+           <inertia ixx="0.01" ixy="0.0" ixz="0.0" iyy="0.01" iyz="0.0" izz="0.01"/>
+       </inertial>
+       <visual>
+           <origin xyz="0 0 0" rpy="0 0 0"/>
+           <geometry>
+               <cylinder radius="0.1" length="0.05"/> <!-- Define as a cylinder for a wheel -->
+           </geometry>
+           <material name="black">
+               <color rgba="0.0 0.0 0.0 1.0"/>
+           </material>
+       </visual>
+       <collision>
+           <origin xyz="0 0 0" rpy="0 0 0"/>
+           <geometry>
+               <cylinder radius="0.1" length="0.05"/>
+           </geometry>
+       </collision>
+   </link>
+   <!-- Wheel 2 Definition -->
+   <link name="wheel2">
+       <inertial>
+           <mass value="1.0"/> <!-- Adjust mass as needed -->
+           <inertia ixx="0.01" ixy="0.0" ixz="0.0" iyy="0.01" iyz="0.0" izz="0.01"/>
+       </inertial>
+       <visual>
+           <origin xyz="0 0 0" rpy="0 0 0"/>
+           <geometry>
+               <cylinder radius="0.1" length="0.05"/>
+           </geometry>
+           <material name="black">
+               <color rgba="0.0 0.0 0.0 1.0"/>
+           </material>
+       </visual>
+       <collision>
+           <origin xyz="0 0 0" rpy="0 0 0"/>
+           <geometry>
+               <cylinder radius="0.1" length="0.05"/>
+           </geometry>
+       </collision>
+   </link>
+   <!-- Wheel 3 Definition -->
+   <link name="wheel3">
+       <inertial>
+           <mass value="1.0"/> <!-- Adjust mass as needed -->
+           <inertia ixx="0.01" ixy="0.0" ixz="0.0" iyy="0.01" iyz="0.0" izz="0.01"/>
+       </inertial>
+       <visual>
+           <origin xyz="0 0 0" rpy="0 0 0"/>
+           <geometry>
+               <cylinder radius="0.1" length="0.05"/>
+           </geometry>
+           <material name="black">
+               <color rgba="0.0 0.0 0.0 1.0"/>
+           </material>
+       </visual>
+       <collision>
+           <origin xyz="0 0 0" rpy="0 0 0"/>
+           <geometry>
+               <cylinder radius="0.1" length="0.05"/>
+           </geometry>
+       </collision>
+   </link>
+   <!-- Joint Definitions for Wheels -->
+   <!-- Joint 1 -->
+   <joint name="wheel1_joint" type="revolute">
+       <parent link="base_link"/> <!-- Connecting to the base link -->
+       <child link="wheel1"/>
+       <origin xyz="0.5 0.5 0.0" rpy="0 0 0"/> <!-- Adjust position to where the wheel should connect on the base -->
+       <axis xyz="0 0 1"/> <!-- Assuming rotation around Z-axis -->
+       <limit lower="-1.57" upper="1.57" effort="10.0" velocity="5.0"/>
+   </joint>
+   <!-- Joint 2 -->
+   <joint name="wheel2_joint" type="revolute">
+       <parent link="base_link"/>
+       <child link="wheel2"/>
+       <origin xyz="0.5 -0.5 0.0" rpy="0 0 0"/> <!-- Adjust position accordingly -->
+       <axis xyz="0 0 1"/>
+       <limit lower="-1.57" upper="1.57" effort="10.0" velocity="5.0"/>
+   </joint>
+   <!-- Joint 3 -->
+   <joint name="wheel3_joint" type="revolute">
+       <parent link="base_link"/>
+       <child link="wheel3"/>
+       <origin xyz="-0.5 0.0 0.0" rpy="0 0 0"/> <!-- Adjust position accordingly -->
+       <axis xyz="0 0 1"/>
+       <limit lower="-1.57" upper="1.57" effort="10.0" velocity="5.0"/>
+   </joint>
+  <gazebo>
+    <plugin name="omni_drive_plugin" filename="libgazebo_ros_skid_steer_drive.so">
+      <ros>
+        <namespace>/robot</namespace>
+        <remapping>cmd_vel:=/cmd_vel</remapping>
+        <remapping>odom:=/odom</remapping>
+      </ros>
+      <updateRate>50.0</updateRate>
+      <!-- Joint names for omni-drive wheels -->
+      <leftJoint>wheel1_joint</leftJoint>
+      <leftJoint>wheel2_joint</leftJoint>
+      <leftJoint>wheel3_joint</leftJoint>
+      <!-- Physical parameters -->
+      <wheelSeparation>0.5</wheelSeparation>
+      <wheelRadius>0.1</wheelRadius>
+      <wheelTorque>1.0</wheelTorque>
+      <!-- Odometry -->
+      <odometryFrame>odom</odometryFrame>
+      <robotBaseFrame>base_link</robotBaseFrame>
+    </plugin>
+  </gazebo>
   <link name="TriOrb300P100_TopPlate">
     <inertial>
