Commit message: bot spawned in simulation

File: warehouse_robot_sim/urdf/TriBot_Oakd.urdf.xacro (robot description, xacro)
@@ -1,4 +1,5 @@
 <?xml version="1.0" ?>
-<robot name="TriOrb300P100_Corrected">
+<robot name="TriOrb300P100">
+  <!-- <xacro:include filename="$(find warehouse_robot_sim)/urdf/oakd.xacro" /> -->
   <link name="base_link">
     <inertial>
@@ -10,5 +11,5 @@
         <origin xyz="0.0 0.0 0.0" rpy="0.0 0.0 0.0" />
         <geometry>
-            <mesh filename="~/tribot/src/warehouse_robot_sim/meshes/TriOrb300P100_UnderPlate.stl" scale="0.001 0.001 0.001" />
+            <mesh filename="file://$(find warehouse_robot_sim)/meshes/TriOrb300P100_UnderPlate.stl" scale="0.001 0.001 0.001" />
         </geometry>
         <material name="sus">
@@ -19,5 +20,5 @@
         <origin xyz="0.0 0.0 0.0" rpy="0.0 0.0 0.0" />
         <geometry>
-            <mesh filename="~/tribot/src/warehouse_robot_sim/meshes/TriOrb300P100_UnderPlate.stl" scale="0.001 0.001 0.001" />
+            <mesh filename="file://$(find warehouse_robot_sim)/meshes/TriOrb300P100_UnderPlate.stl" scale="0.001 0.001 0.001" />
         </geometry>
     </collision>
@@ -32,5 +33,5 @@
         <origin xyz="0.0 0.0 0.0" rpy="0.0 -0.0 0.0" />
         <geometry>
-            <mesh filename="~/tribot/src/warehouse_robot_sim/meshes/TriOrb300P100_TopPlate.stl" scale="0.001 0.001 0.001" />
+            <mesh filename="file://$(find warehouse_robot_sim)/meshes/TriOrb300P100_TopPlate.stl" scale="0.001 0.001 0.001" />
         </geometry>
         <material name="dark_gray">
@@ -41,5 +42,5 @@
         <origin xyz="0.0 0.0 0.0" rpy="0.0 -0.0 0.0" />
         <geometry>
-            <mesh filename="~/tribot/src/warehouse_robot_sim/meshes/TriOrb300P100_TopPlate.stl" scale="0.001 0.001 0.001" />
+            <mesh filename="file://$(find warehouse_robot_sim)/meshes/TriOrb300P100_TopPlate.stl" scale="0.001 0.001 0.001" />
         </geometry>
     </collision>
@@ -139,5 +140,5 @@
         <origin xyz="0.0 -0.131 0.064" rpy="1.5708 0.0 0.0" />
         <geometry>
-            <mesh filename="~/tribot/src/warehouse_robot_sim/meshes/TriOrb300P100_PlateA_PlateA-1.stl" scale="0.001 0.001 0.001" />
+            <mesh filename="file://$(find warehouse_robot_sim)/meshes/TriOrb300P100_PlateA_PlateA-1.stl" scale="0.001 0.001 0.001" />
         </geometry>
         <material name="aluminum">
@@ -148,5 +149,5 @@
         <origin xyz="0.0 -0.131 0.064" rpy="1.5708 0.0 0.0" />
         <geometry>
-            <mesh filename="../meshes/TriOrb300P100_PlateA_PlateA-1.stl" scale="0.001 0.001 0.001" />
+            <mesh filename="file://$(find warehouse_robot_sim)/meshes/TriOrb300P100_PlateA_PlateA-1.stl" scale="0.001 0.001 0.001" />
         </geometry>
     </collision>
@@ -165,5 +166,5 @@
         <origin xyz="0.115 0.067 0.064" rpy="1.5708 0.0 2.0944" />
         <geometry>
-            <mesh filename="~/tribot/src/warehouse_robot_sim/meshes/TriOrb300P100_PlateA_PlateA-1.stl" scale="0.001 0.001 0.001" />
+            <mesh filename="file://$(find warehouse_robot_sim)/meshes/TriOrb300P100_PlateA_PlateA-1.stl" scale="0.001 0.001 0.001" />
         </geometry>
         <material name="aluminum">
@@ -174,5 +175,5 @@
         <origin xyz="0.115 0.067 0.064" rpy="1.5708 0.0 2.0944" />
         <geometry>
-            <mesh filename="~/tribot/src/warehouse_robot_sim/meshes/TriOrb300P100_PlateA_PlateA-1.stl" scale="0.001 0.001 0.001" />
+            <mesh filename="file://$(find warehouse_robot_sim)/meshes/TriOrb300P100_PlateA_PlateA-1.stl" scale="0.001 0.001 0.001" />
         </geometry>
     </collision>
@@ -186,5 +187,5 @@
         <origin xyz="-0.115 0.067 0.064" rpy="1.5708 0.0 -2.0944" />
         <geometry>
-            <mesh filename="~/tribot/src/warehouse_robot_sim/meshes/TriOrb300P100_PlateA_PlateA-1.stl" scale="0.001 0.001 0.001" />
+            <mesh filename="file://$(find warehouse_robot_sim)/meshes/TriOrb300P100_PlateA_PlateA-1.stl" scale="0.001 0.001 0.001" />
         </geometry>
         <material name="aluminum">
@@ -195,5 +196,5 @@
         <origin xyz="-0.115 0.067 0.064" rpy="1.5708 0.0 -2.0944" />
         <geometry>
-            <mesh filename="~/tribot/src/warehouse_robot_sim/meshes/TriOrb300P100_PlateA_PlateA-1.stl" scale="0.001 0.001 0.001" />
+            <mesh filename="file://$(find warehouse_robot_sim)/meshes/TriOrb300P100_PlateA_PlateA-1.stl" scale="0.001 0.001 0.001" />
         </geometry>
     </collision>
@@ -218,5 +219,5 @@
             <origin xyz="0.0 0.226 0.138" rpy="0.0 3.1415 -1.5708" />
             <geometry>
-                <mesh filename="~/tribot/src/warehouse_robot_sim/meshes/TriOrb300P100_Casters_BlockC_BlockC1.stl" scale="0.001 0.001 0.001" />
+                <mesh filename="file://$(find warehouse_robot_sim)/meshes/TriOrb300P100_Casters_BlockC_BlockC1.stl" scale="0.001 0.001 0.001" />
             </geometry>
             <material name="dark_gray">
@@ -227,5 +228,5 @@
             <origin xyz="0.0 0.226 0.138" rpy="0.0 3.1415 -1.5708" />
             <geometry>
-                <mesh filename="~/tribot/src/warehouse_robot_sim/meshes/TriOrb300P100_Casters_BlockC_BlockC1.stl" scale="0.001 0.001 0.001" />
+                <mesh filename="file://$(find warehouse_robot_sim)/meshes/TriOrb300P100_Casters_BlockC_BlockC1.stl" scale="0.001 0.001 0.001" />
             </geometry>
         </collision>
@@ -240,5 +241,5 @@
             <origin xyz="-0.196 -0.113 0.138" rpy="0.0 3.1415 0.521" />
             <geometry>
-                <mesh filename="~/tribot/src/warehouse_robot_sim/meshes/TriOrb300P100_Casters_BlockC_BlockC1.stl" scale="0.001 0.001 0.001" />
+                <mesh filename="file://$(find warehouse_robot_sim)/meshes/TriOrb300P100_Casters_BlockC_BlockC1.stl" scale="0.001 0.001 0.001" />
             </geometry>
             <material name="dark_gray">
@@ -249,5 +250,5 @@
             <origin xyz="-0.196 -0.113 0.138" rpy="0.0 3.1415 0.521" />
             <geometry>
-                <mesh filename="~/tribot/src/warehouse_robot_sim/meshes/TriOrb300P100_Casters_BlockC_BlockC1.stl" scale="0.001 0.001 0.001" />
+                <mesh filename="file://$(find warehouse_robot_sim)/meshes/TriOrb300P100_Casters_BlockC_BlockC1.stl" scale="0.001 0.001 0.001" />
             </geometry>
         </collision>
@@ -262,5 +263,5 @@
             <origin xyz="0.196 -0.113 0.138" rpy="0.0 3.1415 2.6154" />
             <geometry>
-                <mesh filename="~/tribot/src/warehouse_robot_sim/meshes/TriOrb300P100_Casters_BlockC_BlockC1.stl" scale="0.001 0.001 0.001" />
+                <mesh filename="file://$(find warehouse_robot_sim)/meshes/TriOrb300P100_Casters_BlockC_BlockC1.stl" scale="0.001 0.001 0.001" />
             </geometry>
             <material name="dark_gray">
@@ -271,5 +272,5 @@
             <origin xyz="0.196 -0.113 0.138" rpy="0.0 3.1415 2.6154" />
             <geometry>
-                <mesh filename="~/tribot/src/warehouse_robot_sim/meshes/TriOrb300P100_Casters_BlockC_BlockC1.stl" scale="0.001 0.001 0.001" />
+                <mesh filename="file://$(find warehouse_robot_sim)/meshes/TriOrb300P100_Casters_BlockC_BlockC1.stl" scale="0.001 0.001 0.001" />
             </geometry>
         </collision>
@@ -299,5 +300,5 @@
             <origin xyz="-0.057 0.222 0.138" rpy="0 3.1415 2.617901" />
             <geometry>
-                <mesh filename="~/tribot/src/warehouse_robot_sim/meshes/TriOrb300P100_Casters_BlockC_Pall.stl" scale="0.001 0.001 0.001" />
+                <mesh filename="file://$(find warehouse_robot_sim)/meshes/TriOrb300P100_Casters_BlockC_Pall.stl" scale="0.001 0.001 0.001" />
             </geometry>
             <material name="dark_gray">
@@ -308,5 +309,5 @@
             <origin xyz="-0.057 0.222 0.138" rpy="0 3.1415 2.617901" />
             <geometry>
-                <mesh filename="~/tribot/src/warehouse_robot_sim/meshes/TriOrb300P100_Casters_BlockC_Pall.stl" scale="0.001 0.001 0.001" />
+                <mesh filename="file://$(find warehouse_robot_sim)/meshes/TriOrb300P100_Casters_BlockC_Pall.stl" scale="0.001 0.001 0.001" />
             </geometry>
         </collision>
@@ -321,5 +322,5 @@
             <origin xyz="0.057 0.222 0.138" rpy="0 3.1415 0.523599" />
             <geometry>
-                <mesh filename="~/tribot/src/warehouse_robot_sim/meshes/TriOrb300P100_Casters_BlockC_Pall.stl" scale="0.001 0.001 0.001" />
+                <mesh filename="file://$(find warehouse_robot_sim)/meshes/TriOrb300P100_Casters_BlockC_Pall.stl" scale="0.001 0.001 0.001" />
             </geometry>
             <material name="dark_gray">
@@ -330,5 +331,5 @@
             <origin xyz="0.057 0.222 0.138" rpy="0 3.1415 0.523599" />
             <geometry>
-                <mesh filename="~/tribot/src/warehouse_robot_sim/meshes/TriOrb300P100_Casters_BlockC_Pall.stl" scale="0.001 0.001 0.001" />
+                <mesh filename="file://$(find warehouse_robot_sim)/meshes/TriOrb300P100_Casters_BlockC_Pall.stl" scale="0.001 0.001 0.001" />
             </geometry>
         </collision>
@@ -343,5 +344,5 @@
             <origin xyz="0.221 -0.062 0.138" rpy="0 3.1415 0.521" />
             <geometry>
-                <mesh filename="~/tribot/src/warehouse_robot_sim/meshes/TriOrb300P100_Casters_BlockC_Pall.stl" scale="0.001 0.001 0.001" />
+                <mesh filename="file://$(find warehouse_robot_sim)/meshes/TriOrb300P100_Casters_BlockC_Pall.stl" scale="0.001 0.001 0.001" />
             </geometry>
             <material name="dark_gray">
@@ -352,5 +353,5 @@
             <origin xyz="0.221 -0.062 0.138" rpy="0 3.1415 0.521" />
             <geometry>
-                <mesh filename="~/tribot/src/warehouse_robot_sim/meshes/TriOrb300P100_Casters_BlockC_Pall.stl" scale="0.001 0.001 0.001" />
+                <mesh filename="file://$(find warehouse_robot_sim)/meshes/TriOrb300P100_Casters_BlockC_Pall.stl" scale="0.001 0.001 0.001" />
             </geometry>
         </collision>
@@ -365,5 +366,5 @@
             <origin xyz="0.164 -0.16 0.138" rpy="0 3.1415 -1.5734" />
             <geometry>
-                <mesh filename="~/tribot/src/warehouse_robot_sim/meshes/TriOrb300P100_Casters_BlockC_Pall.stl" scale="0.001 0.001 0.001" />
+                <mesh filename="file://$(find warehouse_robot_sim)/meshes/TriOrb300P100_Casters_BlockC_Pall.stl" scale="0.001 0.001 0.001" />
             </geometry>
             <material name="dark_gray">
@@ -374,5 +375,5 @@
             <origin xyz="0.164 -0.16 0.138" rpy="0 3.1415 -1.5734" />
             <geometry>
-                <mesh filename="~/tribot/src/warehouse_robot_sim/meshes/TriOrb300P100_Casters_BlockC_Pall.stl" scale="0.001 0.001 0.001" />
+                <mesh filename="file://$(find warehouse_robot_sim)/meshes/TriOrb300P100_Casters_BlockC_Pall.stl" scale="0.001 0.001 0.001" />
             </geometry>
         </collision>
@@ -387,5 +388,5 @@
             <origin xyz="-0.221 -0.062 0.138" rpy="0 3.1415 2.6154" />
             <geometry>
-                <mesh filename="~/tribot/src/warehouse_robot_sim/meshes/TriOrb300P100_Casters_BlockC_Pall.stl" scale="0.001 0.001 0.001" />
+                <mesh filename="file://$(find warehouse_robot_sim)/meshes/TriOrb300P100_Casters_BlockC_Pall.stl" scale="0.001 0.001 0.001" />
             </geometry>
             <material name="dark_gray">
@@ -396,5 +397,5 @@
             <origin xyz="-0.221 -0.062 0.138" rpy="0 3.1415 2.6154" />
             <geometry>
-                <mesh filename="~/tribot/src/warehouse_robot_sim/meshes/TriOrb300P100_Casters_BlockC_Pall.stl" scale="0.001 0.001 0.001" />
+                <mesh filename="file://$(find warehouse_robot_sim)/meshes/TriOrb300P100_Casters_BlockC_Pall.stl" scale="0.001 0.001 0.001" />
             </geometry>
         </collision>
@@ -409,5 +410,5 @@
             <origin xyz="-0.164 -0.16 0.138" rpy="0 3.1415 4.9715" />
             <geometry>
-                <mesh filename="~/tribot/src/warehouse_robot_sim/meshes/TriOrb300P100_Casters_BlockC_Pall.stl" scale="0.001 0.001 0.001" />
+                <mesh filename="file://$(find warehouse_robot_sim)/meshes/TriOrb300P100_Casters_BlockC_Pall.stl" scale="0.001 0.001 0.001" />
             </geometry>
             <material name="dark_gray">
@@ -418,5 +419,5 @@
             <origin xyz="-0.164 -0.16 0.138" rpy="0 3.1415 4.9715" />
             <geometry>
-                <mesh filename="~/tribot/src/warehouse_robot_sim/meshes/TriOrb300P100_Casters_BlockC_Pall.stl" scale="0.001 0.001 0.001" />
+                <mesh filename="file://$(find warehouse_robot_sim)/meshes/TriOrb300P100_Casters_BlockC_Pall.stl" scale="0.001 0.001 0.001" />
             </geometry>
         </collision>
@@ -461,5 +462,5 @@
             <origin xyz="-0.012 -0.133 0.07" rpy="0.0 0.0 -1.5708" />
             <geometry>
-                <mesh filename="~/tribot/src/warehouse_robot_sim/meshes/TriOrb300P100_PlateA_BLMR5100K-10-B_GPA28GT5150-A-N18.stl" scale="0.001 0.001 0.001" />
+                <mesh filename="file://$(find warehouse_robot_sim)/meshes/TriOrb300P100_PlateA_BLMR5100K-10-B_GPA28GT5150-A-N18.stl" scale="0.001 0.001 0.001" />
             </geometry>
             <material name="white_aluminum">
@@ -470,5 +471,5 @@
             <origin xyz="-0.012 -0.133 0.07" rpy="0.0 0.0 -1.5708" />
             <geometry>
-                <mesh filename="~/tribot/src/warehouse_robot_sim/meshes/TriOrb300P100_PlateA_BLMR5100K-10-B_GPA28GT5150-A-N18.stl" scale="0.001 0.001 0.001" />
+                <mesh filename="file://$(find warehouse_robot_sim)/meshes/TriOrb300P100_PlateA_BLMR5100K-10-B_GPA28GT5150-A-N18.stl" scale="0.001 0.001 0.001" />
             </geometry>
         </collision>
@@ -483,5 +484,5 @@
             <origin xyz="-0.012 -0.123 0.07" rpy="-1.5708 0.0 -1.5708" />
             <geometry>
-                <mesh filename="~/tribot/src/warehouse_robot_sim/meshes/TriOrb300P100_PlateA_BLMR5100K-10-B_Motor.stl" scale="0.001 0.001 0.001" />
+                <mesh filename="file://$(find warehouse_robot_sim)/meshes/TriOrb300P100_PlateA_BLMR5100K-10-B_Motor.stl" scale="0.001 0.001 0.001" />
             </geometry>
             <material name="light_gray">
@@ -492,5 +493,5 @@
             <origin xyz="-0.012 -0.123 0.07" rpy="-1.5708 0.0 -1.5708" />
             <geometry>
-                <mesh filename="~/tribot/src/warehouse_robot_sim/meshes/TriOrb300P100_PlateA_BLMR5100K-10-B_Motor.stl" scale="0.001 0.001 0.001" />
+                <mesh filename="file://$(find warehouse_robot_sim)/meshes/TriOrb300P100_PlateA_BLMR5100K-10-B_Motor.stl" scale="0.001 0.001 0.001" />
             </geometry>
         </collision>
@@ -505,5 +506,5 @@
             <origin xyz="0.123 0.057 0.067" rpy="0.0 0.0 0.523599" />
             <geometry>
-                <mesh filename="~/tribot/src/warehouse_robot_sim/meshes/TriOrb300P100_PlateA_BLMR5100K-10-B_GPA28GT5150-A-N18.stl" scale="0.001 0.001 0.001" />
+                <mesh filename="file://$(find warehouse_robot_sim)/meshes/TriOrb300P100_PlateA_BLMR5100K-10-B_GPA28GT5150-A-N18.stl" scale="0.001 0.001 0.001" />
             </geometry>
             <material name="white_aluminum">
@@ -514,5 +515,5 @@
             <origin xyz="0.123 0.057 0.067" rpy="0.0 0.0 0.523599" />
             <geometry>
-                <mesh filename="~/tribot/src/warehouse_robot_sim/meshes/TriOrb300P100_PlateA_BLMR5100K-10-B_GPA28GT5150-A-N18.stl" scale="0.001 0.001 0.001" />
+                <mesh filename="file://$(find warehouse_robot_sim)/meshes/TriOrb300P100_PlateA_BLMR5100K-10-B_GPA28GT5150-A-N18.stl" scale="0.001 0.001 0.001" />
             </geometry>
         </collision>
@@ -527,5 +528,5 @@
             <origin xyz="0.115 0.052 0.067" rpy="-1.5708 0.0 0.523599" />
             <geometry>
-                <mesh filename="~/tribot/src/warehouse_robot_sim/meshes/TriOrb300P100_PlateA_BLMR5100K-10-B_Motor.stl" scale="0.001 0.001 0.001" />
+                <mesh filename="file://$(find warehouse_robot_sim)/meshes/TriOrb300P100_PlateA_BLMR5100K-10-B_Motor.stl" scale="0.001 0.001 0.001" />
             </geometry>
             <material name="light_gray">
@@ -536,5 +537,5 @@
             <origin xyz="0.115 0.052 0.067" rpy="-1.5708 0.0 0.523599" />
             <geometry>
-                <mesh filename="~/tribot/src/warehouse_robot_sim/meshes/TriOrb300P100_PlateA_BLMR5100K-10-B_Motor.stl" scale="0.001 0.001 0.001" />
+                <mesh filename="file://$(find warehouse_robot_sim)/meshes/TriOrb300P100_PlateA_BLMR5100K-10-B_Motor.stl" scale="0.001 0.001 0.001" />
             </geometry>
         </collision>
@@ -549,5 +550,5 @@
             <origin xyz="-0.111 0.078 0.067" rpy="0.0 0.0 2.61799" />
             <geometry>
-                <mesh filename="~/tribot/src/warehouse_robot_sim/meshes/TriOrb300P100_PlateA_BLMR5100K-10-B_GPA28GT5150-A-N18.stl" scale="0.001 0.001 0.001" />
+                <mesh filename="file://$(find warehouse_robot_sim)/meshes/TriOrb300P100_PlateA_BLMR5100K-10-B_GPA28GT5150-A-N18.stl" scale="0.001 0.001 0.001" />
             </geometry>
             <material name="white_aluminum">
@@ -558,5 +559,5 @@
             <origin xyz="-0.111 0.078 0.067" rpy="0.0 0.0 2.61799" />
             <geometry>
-                <mesh filename="~/tribot/src/warehouse_robot_sim/meshes/TriOrb300P100_PlateA_BLMR5100K-10-B_GPA28GT5150-A-N18.stl" scale="0.001 0.001 0.001" />
+                <mesh filename="file://$(find warehouse_robot_sim)/meshes/TriOrb300P100_PlateA_BLMR5100K-10-B_GPA28GT5150-A-N18.stl" scale="0.001 0.001 0.001" />
             </geometry>
         </collision>
@@ -571,5 +572,5 @@
             <origin xyz="-0.103 0.073 0.067" rpy="-1.5708 0.0 2.61799" />
             <geometry>
-                <mesh filename="~/tribot/src/warehouse_robot_sim/meshes/TriOrb300P100_PlateA_BLMR5100K-10-B_Motor.stl" scale="0.001 0.001 0.001" />
+                <mesh filename="file://$(find warehouse_robot_sim)/meshes/TriOrb300P100_PlateA_BLMR5100K-10-B_Motor.stl" scale="0.001 0.001 0.001" />
             </geometry>
             <material name="light_gray">
@@ -580,5 +581,5 @@
             <origin xyz="-0.103 0.073 0.067" rpy="-1.5708 0.0 2.61799" />
             <geometry>
-                <mesh filename="~/tribot/src/warehouse_robot_sim/meshes/TriOrb300P100_PlateA_BLMR5100K-10-B_Motor.stl" scale="0.001 0.001 0.001" />
+                <mesh filename="file://$(find warehouse_robot_sim)/meshes/TriOrb300P100_PlateA_BLMR5100K-10-B_Motor.stl" scale="0.001 0.001 0.001" />
             </geometry>
         </collision>
@@ -623,5 +624,5 @@
             <origin xyz="0.0 -0.131 0.064" rpy="1.5708 0.0 0.0" />
             <geometry>
-                <mesh filename="~/tribot/src/warehouse_robot_sim/meshes/TriOrb300P100_PlateA_Belt.stl" scale="0.001 0.001 0.001" />
+                <mesh filename="file://$(find warehouse_robot_sim)/meshes/TriOrb300P100_PlateA_Belt.stl" scale="0.001 0.001 0.001" />
             </geometry>
             <material name="black">
@@ -632,5 +633,5 @@
             <origin xyz="0.0 -0.131 0.064" rpy="1.5708 0.0 0.0" />
             <geometry>
-                <mesh filename="~/tribot/src/warehouse_robot_sim/meshes/TriOrb300P100_PlateA_Belt.stl" scale="0.001 0.001 0.001" />
+                <mesh filename="file://$(find warehouse_robot_sim)/meshes/TriOrb300P100_PlateA_Belt.stl" scale="0.001 0.001 0.001" />
             </geometry>
         </collision>
@@ -645,5 +646,5 @@
             <origin xyz="0.115 0.067 0.061" rpy="1.5708 0.0 2.0944" />
             <geometry>
-                <mesh filename="~/tribot/src/warehouse_robot_sim/meshes/TriOrb300P100_PlateA_Belt.stl" scale="0.001 0.001 0.001" />
+                <mesh filename="file://$(find warehouse_robot_sim)/meshes/TriOrb300P100_PlateA_Belt.stl" scale="0.001 0.001 0.001" />
             </geometry>
             <material name="black">
@@ -654,5 +655,5 @@
             <origin xyz="0.115 0.067 0.061" rpy="1.5708 0.0 2.0944" />
             <geometry>
-                <mesh filename="~/tribot/src/warehouse_robot_sim/meshes/TriOrb300P100_PlateA_Belt.stl" scale="0.001 0.001 0.001" />
+                <mesh filename="file://$(find warehouse_robot_sim)/meshes/TriOrb300P100_PlateA_Belt.stl" scale="0.001 0.001 0.001" />
             </geometry>
         </collision>
@@ -667,5 +668,5 @@
             <origin xyz="-0.115 0.067 0.061" rpy="1.5708 0.0 -2.0944" />
             <geometry>
-                <mesh filename="~/tribot/src/warehouse_robot_sim/meshes/TriOrb300P100_PlateA_Belt.stl" scale="0.001 0.001 0.001" />
+                <mesh filename="file://$(find warehouse_robot_sim)/meshes/TriOrb300P100_PlateA_Belt.stl" scale="0.001 0.001 0.001" />
             </geometry>
             <material name="black">
@@ -676,5 +677,5 @@
             <origin xyz="-0.115 0.067 0.061" rpy="1.5708 0.0 -2.0944" />
             <geometry>
-                <mesh filename="~/tribot/src/warehouse_robot_sim/meshes/TriOrb300P100_PlateA_Belt.stl" scale="0.001 0.001 0.001" />
+                <mesh filename="file://$(find warehouse_robot_sim)/meshes/TriOrb300P100_PlateA_Belt.stl" scale="0.001 0.001 0.001" />
             </geometry>
         </collision>
@@ -704,5 +705,5 @@
             <origin xyz="-0.094 -0.153 0.084" rpy="0.0 0.0 1.5708" />
             <geometry>
-                <mesh filename="~/tribot/src/warehouse_robot_sim/meshes/TriOrb300P100_PlateA_Axis_GPA25GT5150-A-N15.stl" scale="0.001 0.001 0.001" />
+                <mesh filename="file://$(find warehouse_robot_sim)/meshes/TriOrb300P100_PlateA_Axis_GPA25GT5150-A-N15.stl" scale="0.001 0.001 0.001" />
             </geometry>
             <material name="white_aluminum">
@@ -713,5 +714,5 @@
             <origin xyz="-0.094 -0.153 0.084" rpy="0.0 0.0 1.5708" />
             <geometry>
-                <mesh filename="~/tribot/src/warehouse_robot_sim/meshes/TriOrb300P100_PlateA_Axis_GPA25GT5150-A-N15.stl" scale="0.001 0.001 0.001" />
+                <mesh filename="file://$(find warehouse_robot_sim)/meshes/TriOrb300P100_PlateA_Axis_GPA25GT5150-A-N15.stl" scale="0.001 0.001 0.001" />
             </geometry>
         </collision>
@@ -726,5 +727,5 @@
             <origin xyz="0.094 -0.153 0.084" rpy="0.0 0.0 1.5708" />
             <geometry>
-                <mesh filename="~/tribot/src/warehouse_robot_sim/meshes/TriOrb300P100_PlateA_Axis_GPA25GT5150-A-N15.stl" scale="0.001 0.001 0.001" />
+                <mesh filename="file://$(find warehouse_robot_sim)/meshes/TriOrb300P100_PlateA_Axis_GPA25GT5150-A-N15.stl" scale="0.001 0.001 0.001" />
             </geometry>
             <material name="white_aluminum">
@@ -735,5 +736,5 @@
             <origin xyz="0.094 -0.153 0.084" rpy="0.0 0.0 1.5708" />
             <geometry>
-                <mesh filename="~/tribot/src/warehouse_robot_sim/meshes/TriOrb300P100_PlateA_Axis_GPA25GT5150-A-N15.stl" scale="0.001 0.001 0.001" />
+                <mesh filename="file://$(find warehouse_robot_sim)/meshes/TriOrb300P100_PlateA_Axis_GPA25GT5150-A-N15.stl" scale="0.001 0.001 0.001" />
             </geometry>
         </collision>
@@ -748,5 +749,5 @@
             <origin xyz="-0.087 0.159 0.081" rpy="0.0 0.0 -0.523599" />
             <geometry>
-                <mesh filename="~/tribot/src/warehouse_robot_sim/meshes/TriOrb300P100_PlateA_Axis_GPA25GT5150-A-N15.stl" scale="0.001 0.001 0.001" />
+                <mesh filename="file://$(find warehouse_robot_sim)/meshes/TriOrb300P100_PlateA_Axis_GPA25GT5150-A-N15.stl" scale="0.001 0.001 0.001" />
             </geometry>
             <material name="white_aluminum">
@@ -757,5 +758,5 @@
             <origin xyz="-0.087 0.159 0.081" rpy="0.0 0.0 -0.523599" />
             <geometry>
-                <mesh filename="~/tribot/src/warehouse_robot_sim/meshes/TriOrb300P100_PlateA_Axis_GPA25GT5150-A-N15.stl" scale="0.001 0.001 0.001" />
+                <mesh filename="file://$(find warehouse_robot_sim)/meshes/TriOrb300P100_PlateA_Axis_GPA25GT5150-A-N15.stl" scale="0.001 0.001 0.001" />
             </geometry>
         </collision>
@@ -770,5 +771,5 @@
             <origin xyz="-0.181 -0.004 0.081" rpy="0.0 0.0 -0.523599" />
             <geometry>
-                <mesh filename="~/tribot/src/warehouse_robot_sim/meshes/TriOrb300P100_PlateA_Axis_GPA25GT5150-A-N15.stl" scale="0.001 0.001 0.001" />
+                <mesh filename="file://$(find warehouse_robot_sim)/meshes/TriOrb300P100_PlateA_Axis_GPA25GT5150-A-N15.stl" scale="0.001 0.001 0.001" />
             </geometry>
             <material name="white_aluminum">
@@ -779,5 +780,5 @@
             <origin xyz="-0.181 -0.004 0.081" rpy="0.0 0.0 -0.523599" />
             <geometry>
-                <mesh filename="~/tribot/src/warehouse_robot_sim/meshes/TriOrb300P100_PlateA_Axis_GPA25GT5150-A-N15.stl" scale="0.001 0.001 0.001" />
+                <mesh filename="file://$(find warehouse_robot_sim)/meshes/TriOrb300P100_PlateA_Axis_GPA25GT5150-A-N15.stl" scale="0.001 0.001 0.001" />
             </geometry>
         </collision>
@@ -792,5 +793,5 @@
             <origin xyz="0.087 0.159 0.081" rpy="0.0 0.0 -2.61799" />
             <geometry>
-                <mesh filename="~/tribot/src/warehouse_robot_sim/meshes/TriOrb300P100_PlateA_Axis_GPA25GT5150-A-N15.stl" scale="0.001 0.001 0.001" />
+                <mesh filename="file://$(find warehouse_robot_sim)/meshes/TriOrb300P100_PlateA_Axis_GPA25GT5150-A-N15.stl" scale="0.001 0.001 0.001" />
             </geometry>
             <material name="white_aluminum">
@@ -801,5 +802,5 @@
             <origin xyz="0.087 0.159 0.081" rpy="0.0 0.0 -2.61799" />
             <geometry>
-                <mesh filename="~/tribot/src/warehouse_robot_sim/meshes/TriOrb300P100_PlateA_Axis_GPA25GT5150-A-N15.stl" scale="0.001 0.001 0.001" />
+                <mesh filename="file://$(find warehouse_robot_sim)/meshes/TriOrb300P100_PlateA_Axis_GPA25GT5150-A-N15.stl" scale="0.001 0.001 0.001" />
             </geometry>
         </collision>
@@ -814,5 +815,5 @@
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