Commit message: bot spawned in simulation

File: warehouse_robot_sim/urdf/oakd.urdf.xacro (robot description, xacro)
@@ -1,5 +1,5 @@
 <?xml version="1.0" ?>
 <!--  xacro macros for oakd mount -->
-<robot name="oakd" xmlns:xacro="http://ros.org/wiki/xacro">
+<robot xmlns:xacro="http://ros.org/wiki/xacro">
       <xacro:macro name="oakd_link" params="mount_point">
       <xacro:property name="oakd_length" value="0.0803" />
@@ -12,5 +12,5 @@
               <origin rpy="0 0 0" xyz="0 0 0" />
               <geometry>
-                      <mesh filename="../meshes/sensors/OAK-D.dae" />
+                      <mesh filename="file://$(find warehouse_robot_sim)/meshes/sensors/OAK-D.dae" />
               </geometry>
                <material name="black" />
@@ -168,5 +168,5 @@
       </gazebo>
     </xacro:macro>
-    <xacro:macro name="oakd_joint" params="x y z roll pitch yaw mount_point" >
+    <!-- <xacro:macro name="oakd_joint" params="x y z roll pitch yaw mount_point" >
         <joint name="oakd_joint_${mount_point}" type="fixed">
                 <origin rpy="${roll} ${pitch} ${yaw}" xyz="${x+0.1} ${y-0.01} ${z}"/>
@@ -177,4 +177,4 @@
             <preserveFixedJoint>true</preserveFixedJoint>
         </gazebo>
-    </xacro:macro>
+    </xacro:macro> -->
 </robot>

Commit message: wheels removed

File: warehouse_robot_sim/urdf/TriBot_Oakd.urdf.xacro (robot description, xacro)
@@ -24,116 +24,4 @@
     </collision>
   </link>
-     <!-- Wheel 1 Definition -->
-   <link name="wheel1">
-       <inertial>
-           <mass value="1.0"/> <!-- Adjust mass as needed -->
-           <inertia ixx="0.01" ixy="0.0" ixz="0.0" iyy="0.01" iyz="0.0" izz="0.01"/>
-       </inertial>
-       <visual>
-           <origin xyz="0 0 0" rpy="0 0 0"/>
-           <geometry>
-               <cylinder radius="0.1" length="0.05"/> <!-- Define as a cylinder for a wheel -->
-           </geometry>
-           <material name="black">
-               <color rgba="0.0 0.0 0.0 1.0"/>
-           </material>
-       </visual>
-       <collision>
-           <origin xyz="0 0 0" rpy="0 0 0"/>
-           <geometry>
-               <cylinder radius="0.1" length="0.05"/>
-           </geometry>
-       </collision>
-   </link>
-   <!-- Wheel 2 Definition -->
-   <link name="wheel2">
-       <inertial>
-           <mass value="1.0"/> <!-- Adjust mass as needed -->
-           <inertia ixx="0.01" ixy="0.0" ixz="0.0" iyy="0.01" iyz="0.0" izz="0.01"/>
-       </inertial>
-       <visual>
-           <origin xyz="0 0 0" rpy="0 0 0"/>
-           <geometry>
-               <cylinder radius="0.1" length="0.05"/>
-           </geometry>
-           <material name="black">
-               <color rgba="0.0 0.0 0.0 1.0"/>
-           </material>
-       </visual>
-       <collision>
-           <origin xyz="0 0 0" rpy="0 0 0"/>
-           <geometry>
-               <cylinder radius="0.1" length="0.05"/>
-           </geometry>
-       </collision>
-   </link>
-   <!-- Wheel 3 Definition -->
-   <link name="wheel3">
-       <inertial>
-           <mass value="1.0"/> <!-- Adjust mass as needed -->
-           <inertia ixx="0.01" ixy="0.0" ixz="0.0" iyy="0.01" iyz="0.0" izz="0.01"/>
-       </inertial>
-       <visual>
-           <origin xyz="0 0 0" rpy="0 0 0"/>
-           <geometry>
-               <cylinder radius="0.1" length="0.05"/>
-           </geometry>
-           <material name="black">
-               <color rgba="0.0 0.0 0.0 1.0"/>
-           </material>
-       </visual>
-       <collision>
-           <origin xyz="0 0 0" rpy="0 0 0"/>
-           <geometry>
-               <cylinder radius="0.1" length="0.05"/>
-           </geometry>
-       </collision>
-   </link>
-   <!-- Joint Definitions for Wheels -->
-   <!-- Joint 1 -->
-   <joint name="wheel1_joint" type="revolute">
-       <parent link="base_link"/> <!-- Connecting to the base link -->
-       <child link="wheel1"/>
-       <origin xyz="0.5 0.5 0.0" rpy="0 0 0"/> <!-- Adjust position to where the wheel should connect on the base -->
-       <axis xyz="0 0 1"/> <!-- Assuming rotation around Z-axis -->
-       <limit lower="-1.57" upper="1.57" effort="10.0" velocity="5.0"/>
-   </joint>
-   <!-- Joint 2 -->
-   <joint name="wheel2_joint" type="revolute">
-       <parent link="base_link"/>
-       <child link="wheel2"/>
-       <origin xyz="0.5 -0.5 0.0" rpy="0 0 0"/> <!-- Adjust position accordingly -->
-       <axis xyz="0 0 1"/>
-       <limit lower="-1.57" upper="1.57" effort="10.0" velocity="5.0"/>
-   </joint>
-   <!-- Joint 3 -->
-   <joint name="wheel3_joint" type="revolute">
-       <parent link="base_link"/>
-       <child link="wheel3"/>
-       <origin xyz="-0.5 0.0 0.0" rpy="0 0 0"/> <!-- Adjust position accordingly -->
-       <axis xyz="0 0 1"/>
-       <limit lower="-1.57" upper="1.57" effort="10.0" velocity="5.0"/>
-   </joint>
-  <gazebo>
-    <plugin name="omni_drive_plugin" filename="libgazebo_ros_skid_steer_drive.so">
-      <ros>
-        <namespace>/robot</namespace>
-        <remapping>cmd_vel:=/cmd_vel</remapping>
-        <remapping>odom:=/odom</remapping>
-      </ros>
-      <updateRate>50.0</updateRate>
-      <!-- Joint names for omni-drive wheels -->
-      <leftJoint>wheel1_joint</leftJoint>
-      <leftJoint>wheel2_joint</leftJoint>
-      <leftJoint>wheel3_joint</leftJoint>
-      <!-- Physical parameters -->
-      <wheelSeparation>0.5</wheelSeparation>
-      <wheelRadius>0.1</wheelRadius>
-      <wheelTorque>1.0</wheelTorque>
-      <!-- Odometry -->
-      <odometryFrame>odom</odometryFrame>
-      <robotBaseFrame>base_link</robotBaseFrame>
-    </plugin>
-  </gazebo>
   <link name="TriOrb300P100_TopPlate">
     <inertial>

Commit message: omnidrive_controller and camera added

File: warehouse_robot_sim/urdf/TriBot_Oakd.urdf.xacro (robot description, xacro)
@@ -1,5 +1,8 @@
 <?xml version="1.0" ?>
-<robot name="TriOrb300P100">
-  <!-- <xacro:include filename="$(find warehouse_robot_sim)/urdf/oakd.urdf.xacro" /> -->
+<robot name="TriOrb300P100" xmlns:xacro="http://ros.org/wiki/xacro">
+  <xacro:include filename="$(find warehouse_robot_sim)/urdf/oakd.urdf.xacro"/>
+  <xacro:include filename="$(find warehouse_robot_sim)/urdf/omni_controller.urdf.xacro" />
+<link name="base_footprint">
+</link>
   <link name="base_link">
     <inertial>
@@ -24,4 +27,9 @@
     </collision>
   </link>
+<joint name="base_joint" type="fixed">
+    <origin xyz="0.0 0.0 0.15" rpy="0.0 0.0 1.57"/>
+    <parent link="base_footprint"/>
+    <child link="base_link"/>
+ </joint>
   <link name="TriOrb300P100_TopPlate">
     <inertial>
@@ -1048,20 +1056,8 @@
   </joint>
   <!--Add camera-->
-  <!-- <xacro:oakd_link mount_point="camera" > -->
-  <!-- </xacro:oakd_link> -->
-  <!-- <xacro:oakd_joint x="0.0" y="0.0" z="0.5" roll="0.0" pitch="0.0" yaw="0.0" mount_point="camera"> -->
-  <!-- </xacro:oakd_joint> -->
+  <xacro:depth_sensor>
+    <origin xyz="0.0 -0.16 0.16" rpy="0.0 0.0 -1.57"/>
+  </xacro:depth_sensor>
       <!-- Add 3-Wheel Omni-Drive Plugin -->
-    <gazebo>
-        <plugin name="omni_drive_plugin" filename="libgazebo_omni_drive_plugin.so">
-            <robot_base_frame>base_link</robot_base_frame>
-            <wheel_radius>0.05</wheel_radius>
-            <wheel_separation>0.3</wheel_separation>
-            <wheel_joints>
-                <joint>TriOrb300P100_Ball100_1_joint</joint>
-                <joint>TriOrb300P100_Ball100_2_joint</joint>
-                <joint>TriOrb300P100_Ball100_3_joint</joint>
-            </wheel_joints>
-        </plugin>
-    </gazebo>
+<xacro:omni_drive_controller />
 </robot>

File: warehouse_robot_sim/urdf/oakd.urdf.xacro (robot description, xacro)
@@ -1,180 +1,90 @@
-<?xml version="1.0" ?>
-<!--  xacro macros for oakd mount -->
 <robot xmlns:xacro="http://ros.org/wiki/xacro">
-      <xacro:macro name="oakd_link" params="mount_point">
-      <xacro:property name="oakd_length" value="0.0803" />
-      <xacro:property name="oakd_width" value="0.0957" />
-      <xacro:property name="oakd_depth" value="0.1267" />
-      <xacro:property name="oakd_mass" value="0.15" />
-      <link name="oakd_${mount_point}">
-             <pose>0.0 0.0 0.0 0.0 0.0 0.0</pose>
-          <visual>
-              <origin rpy="0 0 0" xyz="0 0 0" />
-              <geometry>
-                      <mesh filename="file://$(find warehouse_robot_sim)/meshes/sensors/OAK-D.dae" />
-              </geometry>
-               <material name="black" />
-          </visual>
-          <collision>
-              <origin rpy="0 0 0" xyz="0 0 0" />
-              <geometry>
-                  <box size="${oakd_length} ${oakd_width} ${oakd_depth}"/>
-              </geometry>
-          </collision>
-          <xacro:solid_cuboid_inertial
-              rpy="0 0 0" xyz="0 0 0"
-              mass="${oakd_mass}"
-              x="${oakd_length}" y="${oakd_width}" z="${oakd_depth}" />
-      </link>
-      <!-- Add dummy joint for camera_optical_frame to link back to base_link -->
-      <joint name="camera_optical_joint" type="fixed">
-      <!-- Point cloud frustrum is 90 degrees off from visual frame -->
-           <origin rpy="-1.57079632769 0 -1.570796332769" xyz="0 0 0" />
-	   <parent link="oakd_${mount_point}" />
-	   <child link="camera_optical_frame" />
-	</joint>
-	<!-- Add dummy link for camera_optical_frame to link back to base_link -->
-        <link name="camera_optical_frame">
-        <inertial>
-	  <mass value="0.001" />
-	  <origin xyz="0 0 0" />
-	  <inertia ixx="0.0001" ixy="0.0" ixz="0.0" iyy="0.0001" iyz="0.0" izz="0.0001" />
-          </inertial>
-  </link>
-  <!-- Dummy joints for rgb camera to link back to base_link -->
-        <joint name="camera_rgb_optical_joint" type="fixed">
-           <origin rpy="0 0 0" xyz="0 0 0" />
-	   <parent link="oakd_${mount_point}" />
-	   <child link="camera_rgb_optical_frame" />
-	</joint>
-	<!-- Add dummy link for camera_optical_frame to link back to base_link -->
-        <link name="camera_rgb_optical_frame">
-        <inertial>
-	  <mass value="0.001" />
-	  <origin xyz="0 0 0" />
-	  <inertia ixx="0.0001" ixy="0.0" ixz="0.0" iyy="0.0001" iyz="0.0" izz="0.0001" />
-          </inertial>
-  </link>
-  <!-- Gazebo plugin for greyscale left/right stereo pairs -->
-      <gazebo reference="oakd_${mount_point}">
-    <material>Gazebo/DarkGrey</material>
-    <sensor type="multicamera" name="stereo_camera">
-      <update_rate>30.0</update_rate>
-      <camera name="left">
-        <horizontal_fov>1.2566</horizontal_fov>
-        <image>
-          <width>1200</width>
-          <height>800</height>
-	  <format>L8</format>
-	  <!--   <format>R8G8B8</format> -->
-        </image>
-        <clip>
-          <near>0.3</near>
-          <far>35</far>
-        </clip>
-        <noise>
-          <type>gaussian</type>
-          <mean>0.0</mean>
-          <stddev>0.007</stddev>
-        </noise>
-      </camera>
-      <camera name="right">
-        <pose>0 -0.07 0 0 0 0</pose>
-        <horizontal_fov>1.1.2566</horizontal_fov>
-        <image>
-          <width>1200</width>
-          <height>800</height>
-	  <format>L8</format>
-	  <!--   <format>R8G8B8</format> -->
-        </image>
-        <clip>
-          <near>0.3</near>
-          <far>35</far>
-        </clip>
-        <noise>
-          <type>gaussian</type>
-          <mean>0.0</mean>
-          <stddev>0.007</stddev>
-        </noise>
-      </camera>
-      <plugin name="stereo_camera_controller" filename="libgazebo_ros_multicamera.so">
-        <alwaysOn>true</alwaysOn>
-        <updateRate>0.0</updateRate>
-	<cameraName>oakd_${mount_point}/camera</cameraName>
-        <imageTopicName>image_raw</imageTopicName>
-        <cameraInfoTopicName>camera_info</cameraInfoTopicName>
-	<frameName>camera_optical_frame</frameName>
-        <!--<rightFrameName>right_camera_optical_frame</rightFrameName>-->
-        <hackBaseline>0.075</hackBaseline>
-        <distortionK1>0.0</distortionK1>
-        <distortionK2>0.0</distortionK2>
-        <distortionK3>0.0</distortionK3>
-        <distortionT1>0.0</distortionT1>
-        <distortionT2>0.0</distortionT2>
-      </plugin>
-    </sensor>
-  </gazebo>
- <!-- Gazebo plugin for center RGB camera -->
-   <gazebo reference="oakd_${mount_point}">
-      <material>Gazebo/White</material>
-      <sensor type="camera" name="oakd_rgb_${mount_point}">
-      <update_rate>30.0</update_rate>
-      <camera name="head">
-        <horizontal_fov>1.3962634</horizontal_fov>
-        <image>
-          <width>800</width>
-          <height>800</height>
-          <format>R8G8B8</format>
-        </image>
-        <clip>
-          <near>0.02</near>
-          <far>300</far>
-        </clip>
-        <noise>
-          <type>gaussian</type>
-          <!-- Noise is sampled independently per pixel on each frame.
-               That pixel's noise value is added to each of its color
-               channels, which at that point lie in the range [0,1]. -->
-          <mean>0.0</mean>
-          <stddev>0.007</stddev>
-        </noise>
-      </camera>
-      <plugin name="camera_controller" filename="libgazebo_ros_camera.so">
-        <alwaysOn>true</alwaysOn>
-        <updateRate>0.0</updateRate>
-        <cameraName>oakd_rgb_${mount_point}</cameraName>
-        <imageTopicName>image_raw</imageTopicName>
-        <cameraInfoTopicName>camera_info</cameraInfoTopicName>
-        <frameName>camera_rgb_link_optical</frameName>
-        <!-- setting hackBaseline to anything but 0.0 will cause a misalignment
-            between the gazebo sensor image and the frame it is supposed to
-            be attached to -->
-        <hackBaseline>0.0</hackBaseline>
-        <distortionK1>0.0</distortionK1>
-        <distortionK2>0.0</distortionK2>
-        <distortionK3>0.0</distortionK3>
-        <distortionT1>0.0</distortionT1>
-        <distortionT2>0.0</distortionT2>
-        <CxPrime>0</CxPrime>
-        <Cx>0.0</Cx>
-        <Cy>0.0</Cy>
-        <focalLength>0.0</focalLength>
-      </plugin>
-    </sensor>
-  </gazebo>
-      <gazebo reference="oakd_joint_${mount_point}">
-          <!-- <disableFixedJointLumping>true</disableFixedJointLumping>  -->
-          <!-- <preserveFixedJoint>true</preserveFixedJoint> -->
-      </gazebo>
-    </xacro:macro>
-    <!-- <xacro:macro name="oakd_joint" params="x y z roll pitch yaw mount_point" >
-        <joint name="oakd_joint_${mount_point}" type="fixed">
-                <origin rpy="${roll} ${pitch} ${yaw}" xyz="${x+0.1} ${y-0.01} ${z}"/>
-            <parent link="base_link" />
-            <child link="oakd_${mount_point}" />
-        </joint>
-        <gazebo reference="oakd_joint_${mount_point}">
-            <preserveFixedJoint>true</preserveFixedJoint>
-        </gazebo>
-    </xacro:macro> -->
+  <xacro:property name="M_PI" value="3.1415926535897931" />
+  <xacro:macro name="depth_sensor" params="*origin">
+    <link name="camera_link">
+      <visual>
+        <origin xyz="0 0 0" rpy="0 0 0"/>
+        <geometry>
+          <box size="0.030 0.124 0.030"/>
+          <!-- <mesh filename="" scale="0.001 0.001 0.001"/> -->
+        </geometry>
+        <material name="red">
+          <color rgba="0.416 0.051 0.047 1.0"/>
+        </material>
+      </visual>
+      <collision>
+        <origin xyz="0 0 0" rpy="0 0 0"/>
+        <geometry>
+          <box size="0.030 0.124 0.030"/>
+        </geometry>
+      </collision>
+      <inertial>
+        <origin xyz="0 0 0" rpy="0 0 0"/>
+        <mass value="0.135"/>
+        <inertia ixx="${(1/12) * 0.135 * ((0.124  * 0.124)  + (0.030 * 0.030))}" ixy="0.0" ixz="0.0"
+                 iyy="${(1/12) * 0.135 * ((0.030 * 0.030) + (0.030 * 0.030))}" iyz="0.0"
+                 izz="${(1/12) * 0.135 * ((0.030 * 0.030) + (0.124  * 0.124))}"/>
+      </inertial>
+    </link>
+    <gazebo reference="camera_link">
+      <visual>
+        <material>
+          <ambient>0.416 0.051 0.047 1.0</ambient>
+          <diffuse>0.416 0.051 0.047 1.0</diffuse>
+          <specular>0.416 0.051 0.047 1.0</specular>
+          <emissive>0.416 0.051 0.047 1.0</emissive>
+        </material>
+      </visual>
+    </gazebo>rgb(213,28,40)
+    <joint name="camera_to_base_link" type="fixed">
+      <parent link="base_link"/>
+      <child link="camera_link"/>
+      <xacro:insert_block name="origin" />
+    </joint>
+    <link name="camera_depth_link"/>
+    <joint name="camera_depth_joint" type="fixed">
+      <origin xyz="0 0 0" rpy="-1.57 0 -1.57"/>
+      <parent link="camera_link"/>
+      <child link="camera_depth_link"/>
+    </joint>
+    <!-- https://github.com/ros-simulation/gazebo_ros_pkgs/wiki/ROS-2-Migration:-Camera#gazebo_ros_camera -->
+    <gazebo reference="camera_link">
+      <sensor name="camera" type="depth">
+        <always_on>true</always_on>
+        <update_rate>30.0</update_rate>
+        <camera name="camera">
+          <horizontal_fov>1.50098</horizontal_fov>
+          <image>
+            <width>640</width>
+            <height>480</height>
+            <format>R8G8B8</format>
+          </image>
+        </camera>
+        <plugin name="camera_controller" filename="libgazebo_ros_camera.so">
+          <ros>
+            <remapping>/camera/camera_info:=/camera/color/camera_info</remapping>
+            <remapping>/camera/image_raw:=/camera/color/image_raw</remapping>
+            <remapping>/camera/points:=/camera/depth/color/points</remapping>
+            <remapping>/camera/depth/image_raw:=/camera/depth/image_rect_raw</remapping>
+            <qos>
+              <topic name="/camera/depth/color/points">
+                <publisher>
+                  <reliability>best_effort</reliability>
+                </publisher>
+              </topic>
+            </qos>
+          </ros>
+          <min_depth>0.015</min_depth>
+          <max_depth>3.0</max_depth>
+          <hack_baseline>0.07</hack_baseline>
+          <frame_name>camera_depth_link</frame_name>
+          <distortion_k1>0.00000001</distortion_k1>
+          <distortion_k2>0.00000001</distortion_k2>
+          <distortion_k3>0.00000001</distortion_k3>
+          <distortion_t1>0.00000001</distortion_t1>
+          <distortion_t2>0.00000001</distortion_t2>
+        </plugin>
+      </sensor>
+    </gazebo>
+  </xacro:macro>
 </robot>
