Commit message: Removed config error

File: warehouse_robot_sim/urdf/TriBot_Oakd.urdf.xacro (robot description, xacro)
@@ -1,4 +1,8 @@
 <?xml version="1.0" ?>
-<robot name="TriOrb300P100">
+<robot name="TriOrb300P100" xmlns:xacro="http://ros.org/wiki/xacro">
+  <xacro:include filename="$(find warehouse_robot_sim)/urdf/oakd.urdf.xacro"/>
+  <xacro:include filename="$(find warehouse_robot_sim)/urdf/omni_controller.urdf.xacro" />
+<link name="base_footprint">
+</link>
   <link name="base_link">
     <inertial>
@@ -10,5 +14,5 @@
         <origin xyz="0.0 0.0 0.0" rpy="0.0 0.0 0.0" />
         <geometry>
-            <mesh filename="~/tribot/src/warehouse_robot_sim/meshes/TriOrb300P100_UnderPlate.stl" scale="0.001 0.001 0.001" />
+            <mesh filename="file://$(find warehouse_robot_sim)/meshes/TriOrb300P100_UnderPlate.stl" scale="0.001 0.001 0.001" />
         </geometry>
         <material name="sus">
@@ -19,120 +23,13 @@
         <origin xyz="0.0 0.0 0.0" rpy="0.0 0.0 0.0" />
         <geometry>
-            <mesh filename="~/tribot/src/warehouse_robot_sim/meshes/TriOrb300P100_UnderPlate.stl" scale="0.001 0.001 0.001" />
+            <mesh filename="file://$(find warehouse_robot_sim)/meshes/TriOrb300P100_UnderPlate.stl" scale="0.001 0.001 0.001" />
         </geometry>
     </collision>
   </link>
-     <!-- Wheel 1 Definition -->
-   <link name="wheel1">
-       <inertial>
-           <mass value="1.0"/> <!-- Adjust mass as needed -->
-           <inertia ixx="0.01" ixy="0.0" ixz="0.0" iyy="0.01" iyz="0.0" izz="0.01"/>
-       </inertial>
-       <visual>
-           <origin xyz="0 0 0" rpy="0 0 0"/>
-           <geometry>
-               <cylinder radius="0.1" length="0.05"/> <!-- Define as a cylinder for a wheel -->
-           </geometry>
-           <material name="black">
-               <color rgba="0.0 0.0 0.0 1.0"/>
-           </material>
-       </visual>
-       <collision>
-           <origin xyz="0 0 0" rpy="0 0 0"/>
-           <geometry>
-               <cylinder radius="0.1" length="0.05"/>
-           </geometry>
-       </collision>
-   </link>
-   <!-- Wheel 2 Definition -->
-   <link name="wheel2">
-       <inertial>
-           <mass value="1.0"/> <!-- Adjust mass as needed -->
-           <inertia ixx="0.01" ixy="0.0" ixz="0.0" iyy="0.01" iyz="0.0" izz="0.01"/>
-       </inertial>
-       <visual>
-           <origin xyz="0 0 0" rpy="0 0 0"/>
-           <geometry>
-               <cylinder radius="0.1" length="0.05"/>
-           </geometry>
-           <material name="black">
-               <color rgba="0.0 0.0 0.0 1.0"/>
-           </material>
-       </visual>
-       <collision>
-           <origin xyz="0 0 0" rpy="0 0 0"/>
-           <geometry>
-               <cylinder radius="0.1" length="0.05"/>
-           </geometry>
-       </collision>
-   </link>
-   <!-- Wheel 3 Definition -->
-   <link name="wheel3">
-       <inertial>
-           <mass value="1.0"/> <!-- Adjust mass as needed -->
-           <inertia ixx="0.01" ixy="0.0" ixz="0.0" iyy="0.01" iyz="0.0" izz="0.01"/>
-       </inertial>
-       <visual>
-           <origin xyz="0 0 0" rpy="0 0 0"/>
-           <geometry>
-               <cylinder radius="0.1" length="0.05"/>
-           </geometry>
-           <material name="black">
-               <color rgba="0.0 0.0 0.0 1.0"/>
-           </material>
-       </visual>
-       <collision>
-           <origin xyz="0 0 0" rpy="0 0 0"/>
-           <geometry>
-               <cylinder radius="0.1" length="0.05"/>
-           </geometry>
-       </collision>
-   </link>
-   <!-- Joint Definitions for Wheels -->
-   <!-- Joint 1 -->
-   <joint name="wheel1_joint" type="revolute">
-       <parent link="base_link"/> <!-- Connecting to the base link -->
-       <child link="wheel1"/>
-       <origin xyz="0.5 0.5 0.0" rpy="0 0 0"/> <!-- Adjust position to where the wheel should connect on the base -->
-       <axis xyz="0 0 1"/> <!-- Assuming rotation around Z-axis -->
-       <limit lower="-1.57" upper="1.57" effort="10.0" velocity="5.0"/>
-   </joint>
-   <!-- Joint 2 -->
-   <joint name="wheel2_joint" type="revolute">
-       <parent link="base_link"/>
-       <child link="wheel2"/>
-       <origin xyz="0.5 -0.5 0.0" rpy="0 0 0"/> <!-- Adjust position accordingly -->
-       <axis xyz="0 0 1"/>
-       <limit lower="-1.57" upper="1.57" effort="10.0" velocity="5.0"/>
-   </joint>
-   <!-- Joint 3 -->
-   <joint name="wheel3_joint" type="revolute">
-       <parent link="base_link"/>
-       <child link="wheel3"/>
-       <origin xyz="-0.5 0.0 0.0" rpy="0 0 0"/> <!-- Adjust position accordingly -->
-       <axis xyz="0 0 1"/>
-       <limit lower="-1.57" upper="1.57" effort="10.0" velocity="5.0"/>
-   </joint>
-  <gazebo>
-    <plugin name="omni_drive_plugin" filename="libgazebo_ros_skid_steer_drive.so">
-      <ros>
-        <namespace>/robot</namespace>
-        <remapping>cmd_vel:=/cmd_vel</remapping>
-        <remapping>odom:=/odom</remapping>
-      </ros>
-      <updateRate>50.0</updateRate>
-      <!-- Joint names for omni-drive wheels -->
-      <leftJoint>wheel1_joint</leftJoint>
-      <leftJoint>wheel2_joint</leftJoint>
-      <leftJoint>wheel3_joint</leftJoint>
-      <!-- Physical parameters -->
-      <wheelSeparation>0.5</wheelSeparation>
-      <wheelRadius>0.1</wheelRadius>
-      <wheelTorque>1.0</wheelTorque>
-      <!-- Odometry -->
-      <odometryFrame>odom</odometryFrame>
-      <robotBaseFrame>base_link</robotBaseFrame>
-    </plugin>
-  </gazebo>
+<joint name="base_joint" type="fixed">
+    <origin xyz="0.0 0.0 0.15" rpy="0.0 0.0 1.57"/>
+    <parent link="base_footprint"/>
+    <child link="base_link"/>
+ </joint>
   <link name="TriOrb300P100_TopPlate">
     <inertial>
@@ -144,5 +41,5 @@
         <origin xyz="0.0 0.0 0.0" rpy="0.0 -0.0 0.0" />
         <geometry>
-            <mesh filename="~/tribot/src/warehouse_robot_sim/meshes/TriOrb300P100_TopPlate.stl" scale="0.001 0.001 0.001" />
+            <mesh filename="file://$(find warehouse_robot_sim)/meshes/TriOrb300P100_TopPlate.stl" scale="0.001 0.001 0.001" />
         </geometry>
         <material name="dark_gray">
@@ -153,5 +50,5 @@
         <origin xyz="0.0 0.0 0.0" rpy="0.0 -0.0 0.0" />
         <geometry>
-            <mesh filename="~/tribot/src/warehouse_robot_sim/meshes/TriOrb300P100_TopPlate.stl" scale="0.001 0.001 0.001" />
+            <mesh filename="file://$(find warehouse_robot_sim)/meshes/TriOrb300P100_TopPlate.stl" scale="0.001 0.001 0.001" />
         </geometry>
     </collision>
@@ -251,5 +148,5 @@
         <origin xyz="0.0 -0.131 0.064" rpy="1.5708 0.0 0.0" />
         <geometry>
-            <mesh filename="~/tribot/src/warehouse_robot_sim/meshes/TriOrb300P100_PlateA_PlateA-1.stl" scale="0.001 0.001 0.001" />
+            <mesh filename="file://$(find warehouse_robot_sim)/meshes/TriOrb300P100_PlateA_PlateA-1.stl" scale="0.001 0.001 0.001" />
         </geometry>
         <material name="aluminum">
@@ -260,5 +157,5 @@
         <origin xyz="0.0 -0.131 0.064" rpy="1.5708 0.0 0.0" />
         <geometry>
-            <mesh filename="../meshes/TriOrb300P100_PlateA_PlateA-1.stl" scale="0.001 0.001 0.001" />
+            <mesh filename="file://$(find warehouse_robot_sim)/meshes/TriOrb300P100_PlateA_PlateA-1.stl" scale="0.001 0.001 0.001" />
         </geometry>
     </collision>
@@ -277,5 +174,5 @@
         <origin xyz="0.115 0.067 0.064" rpy="1.5708 0.0 2.0944" />
         <geometry>
-            <mesh filename="~/tribot/src/warehouse_robot_sim/meshes/TriOrb300P100_PlateA_PlateA-1.stl" scale="0.001 0.001 0.001" />
+            <mesh filename="file://$(find warehouse_robot_sim)/meshes/TriOrb300P100_PlateA_PlateA-1.stl" scale="0.001 0.001 0.001" />
         </geometry>
         <material name="aluminum">
@@ -286,5 +183,5 @@
         <origin xyz="0.115 0.067 0.064" rpy="1.5708 0.0 2.0944" />
         <geometry>
-            <mesh filename="~/tribot/src/warehouse_robot_sim/meshes/TriOrb300P100_PlateA_PlateA-1.stl" scale="0.001 0.001 0.001" />
+            <mesh filename="file://$(find warehouse_robot_sim)/meshes/TriOrb300P100_PlateA_PlateA-1.stl" scale="0.001 0.001 0.001" />
         </geometry>
     </collision>
@@ -298,5 +195,5 @@
         <origin xyz="-0.115 0.067 0.064" rpy="1.5708 0.0 -2.0944" />
         <geometry>
-            <mesh filename="~/tribot/src/warehouse_robot_sim/meshes/TriOrb300P100_PlateA_PlateA-1.stl" scale="0.001 0.001 0.001" />
+            <mesh filename="file://$(find warehouse_robot_sim)/meshes/TriOrb300P100_PlateA_PlateA-1.stl" scale="0.001 0.001 0.001" />
         </geometry>
         <material name="aluminum">
@@ -307,5 +204,5 @@
         <origin xyz="-0.115 0.067 0.064" rpy="1.5708 0.0 -2.0944" />
         <geometry>
-            <mesh filename="~/tribot/src/warehouse_robot_sim/meshes/TriOrb300P100_PlateA_PlateA-1.stl" scale="0.001 0.001 0.001" />
+            <mesh filename="file://$(find warehouse_robot_sim)/meshes/TriOrb300P100_PlateA_PlateA-1.stl" scale="0.001 0.001 0.001" />
         </geometry>
     </collision>
@@ -330,5 +227,5 @@
             <origin xyz="0.0 0.226 0.138" rpy="0.0 3.1415 -1.5708" />
             <geometry>
-                <mesh filename="~/tribot/src/warehouse_robot_sim/meshes/TriOrb300P100_Casters_BlockC_BlockC1.stl" scale="0.001 0.001 0.001" />
+                <mesh filename="file://$(find warehouse_robot_sim)/meshes/TriOrb300P100_Casters_BlockC_BlockC1.stl" scale="0.001 0.001 0.001" />
             </geometry>
             <material name="dark_gray">
@@ -339,5 +236,5 @@
             <origin xyz="0.0 0.226 0.138" rpy="0.0 3.1415 -1.5708" />
             <geometry>
-                <mesh filename="~/tribot/src/warehouse_robot_sim/meshes/TriOrb300P100_Casters_BlockC_BlockC1.stl" scale="0.001 0.001 0.001" />
+                <mesh filename="file://$(find warehouse_robot_sim)/meshes/TriOrb300P100_Casters_BlockC_BlockC1.stl" scale="0.001 0.001 0.001" />
             </geometry>
         </collision>
@@ -352,5 +249,5 @@
             <origin xyz="-0.196 -0.113 0.138" rpy="0.0 3.1415 0.521" />
             <geometry>
-                <mesh filename="~/tribot/src/warehouse_robot_sim/meshes/TriOrb300P100_Casters_BlockC_BlockC1.stl" scale="0.001 0.001 0.001" />
+                <mesh filename="file://$(find warehouse_robot_sim)/meshes/TriOrb300P100_Casters_BlockC_BlockC1.stl" scale="0.001 0.001 0.001" />
             </geometry>
             <material name="dark_gray">
@@ -361,5 +258,5 @@
             <origin xyz="-0.196 -0.113 0.138" rpy="0.0 3.1415 0.521" />
             <geometry>
-                <mesh filename="~/tribot/src/warehouse_robot_sim/meshes/TriOrb300P100_Casters_BlockC_BlockC1.stl" scale="0.001 0.001 0.001" />
+                <mesh filename="file://$(find warehouse_robot_sim)/meshes/TriOrb300P100_Casters_BlockC_BlockC1.stl" scale="0.001 0.001 0.001" />
             </geometry>
         </collision>
@@ -374,5 +271,5 @@
             <origin xyz="0.196 -0.113 0.138" rpy="0.0 3.1415 2.6154" />
             <geometry>
-                <mesh filename="~/tribot/src/warehouse_robot_sim/meshes/TriOrb300P100_Casters_BlockC_BlockC1.stl" scale="0.001 0.001 0.001" />
+                <mesh filename="file://$(find warehouse_robot_sim)/meshes/TriOrb300P100_Casters_BlockC_BlockC1.stl" scale="0.001 0.001 0.001" />
             </geometry>
             <material name="dark_gray">
@@ -383,5 +280,5 @@
             <origin xyz="0.196 -0.113 0.138" rpy="0.0 3.1415 2.6154" />
             <geometry>
-                <mesh filename="~/tribot/src/warehouse_robot_sim/meshes/TriOrb300P100_Casters_BlockC_BlockC1.stl" scale="0.001 0.001 0.001" />
+                <mesh filename="file://$(find warehouse_robot_sim)/meshes/TriOrb300P100_Casters_BlockC_BlockC1.stl" scale="0.001 0.001 0.001" />
             </geometry>
         </collision>
@@ -411,5 +308,5 @@
             <origin xyz="-0.057 0.222 0.138" rpy="0 3.1415 2.617901" />
             <geometry>
-                <mesh filename="~/tribot/src/warehouse_robot_sim/meshes/TriOrb300P100_Casters_BlockC_Pall.stl" scale="0.001 0.001 0.001" />
+                <mesh filename="file://$(find warehouse_robot_sim)/meshes/TriOrb300P100_Casters_BlockC_Pall.stl" scale="0.001 0.001 0.001" />
             </geometry>
             <material name="dark_gray">
@@ -420,5 +317,5 @@
             <origin xyz="-0.057 0.222 0.138" rpy="0 3.1415 2.617901" />
             <geometry>
-                <mesh filename="~/tribot/src/warehouse_robot_sim/meshes/TriOrb300P100_Casters_BlockC_Pall.stl" scale="0.001 0.001 0.001" />
+                <mesh filename="file://$(find warehouse_robot_sim)/meshes/TriOrb300P100_Casters_BlockC_Pall.stl" scale="0.001 0.001 0.001" />
             </geometry>
         </collision>
@@ -433,5 +330,5 @@
             <origin xyz="0.057 0.222 0.138" rpy="0 3.1415 0.523599" />
             <geometry>
-                <mesh filename="~/tribot/src/warehouse_robot_sim/meshes/TriOrb300P100_Casters_BlockC_Pall.stl" scale="0.001 0.001 0.001" />
+                <mesh filename="file://$(find warehouse_robot_sim)/meshes/TriOrb300P100_Casters_BlockC_Pall.stl" scale="0.001 0.001 0.001" />
             </geometry>
             <material name="dark_gray">
@@ -442,5 +339,5 @@
             <origin xyz="0.057 0.222 0.138" rpy="0 3.1415 0.523599" />
             <geometry>
-                <mesh filename="~/tribot/src/warehouse_robot_sim/meshes/TriOrb300P100_Casters_BlockC_Pall.stl" scale="0.001 0.001 0.001" />
+                <mesh filename="file://$(find warehouse_robot_sim)/meshes/TriOrb300P100_Casters_BlockC_Pall.stl" scale="0.001 0.001 0.001" />
             </geometry>
         </collision>
@@ -455,5 +352,5 @@
             <origin xyz="0.221 -0.062 0.138" rpy="0 3.1415 0.521" />
             <geometry>
-                <mesh filename="~/tribot/src/warehouse_robot_sim/meshes/TriOrb300P100_Casters_BlockC_Pall.stl" scale="0.001 0.001 0.001" />
+                <mesh filename="file://$(find warehouse_robot_sim)/meshes/TriOrb300P100_Casters_BlockC_Pall.stl" scale="0.001 0.001 0.001" />
             </geometry>
             <material name="dark_gray">
@@ -464,5 +361,5 @@
             <origin xyz="0.221 -0.062 0.138" rpy="0 3.1415 0.521" />
             <geometry>
-                <mesh filename="~/tribot/src/warehouse_robot_sim/meshes/TriOrb300P100_Casters_BlockC_Pall.stl" scale="0.001 0.001 0.001" />
+                <mesh filename="file://$(find warehouse_robot_sim)/meshes/TriOrb300P100_Casters_BlockC_Pall.stl" scale="0.001 0.001 0.001" />
             </geometry>
         </collision>
@@ -477,5 +374,5 @@
             <origin xyz="0.164 -0.16 0.138" rpy="0 3.1415 -1.5734" />
             <geometry>
-                <mesh filename="~/tribot/src/warehouse_robot_sim/meshes/TriOrb300P100_Casters_BlockC_Pall.stl" scale="0.001 0.001 0.001" />
+                <mesh filename="file://$(find warehouse_robot_sim)/meshes/TriOrb300P100_Casters_BlockC_Pall.stl" scale="0.001 0.001 0.001" />
             </geometry>
             <material name="dark_gray">
@@ -486,5 +383,5 @@
             <origin xyz="0.164 -0.16 0.138" rpy="0 3.1415 -1.5734" />
             <geometry>
-                <mesh filename="~/tribot/src/warehouse_robot_sim/meshes/TriOrb300P100_Casters_BlockC_Pall.stl" scale="0.001 0.001 0.001" />
+                <mesh filename="file://$(find warehouse_robot_sim)/meshes/TriOrb300P100_Casters_BlockC_Pall.stl" scale="0.001 0.001 0.001" />
             </geometry>
         </collision>
@@ -499,5 +396,5 @@
             <origin xyz="-0.221 -0.062 0.138" rpy="0 3.1415 2.6154" />
             <geometry>
-                <mesh filename="~/tribot/src/warehouse_robot_sim/meshes/TriOrb300P100_Casters_BlockC_Pall.stl" scale="0.001 0.001 0.001" />
+                <mesh filename="file://$(find warehouse_robot_sim)/meshes/TriOrb300P100_Casters_BlockC_Pall.stl" scale="0.001 0.001 0.001" />
             </geometry>
             <material name="dark_gray">
@@ -508,5 +405,5 @@
             <origin xyz="-0.221 -0.062 0.138" rpy="0 3.1415 2.6154" />
             <geometry>
-                <mesh filename="~/tribot/src/warehouse_robot_sim/meshes/TriOrb300P100_Casters_BlockC_Pall.stl" scale="0.001 0.001 0.001" />
+                <mesh filename="file://$(find warehouse_robot_sim)/meshes/TriOrb300P100_Casters_BlockC_Pall.stl" scale="0.001 0.001 0.001" />
             </geometry>
         </collision>
@@ -521,5 +418,5 @@
             <origin xyz="-0.164 -0.16 0.138" rpy="0 3.1415 4.9715" />
             <geometry>
-                <mesh filename="~/tribot/src/warehouse_robot_sim/meshes/TriOrb300P100_Casters_BlockC_Pall.stl" scale="0.001 0.001 0.001" />
+                <mesh filename="file://$(find warehouse_robot_sim)/meshes/TriOrb300P100_Casters_BlockC_Pall.stl" scale="0.001 0.001 0.001" />
             </geometry>
             <material name="dark_gray">
@@ -530,5 +427,5 @@
             <origin xyz="-0.164 -0.16 0.138" rpy="0 3.1415 4.9715" />
             <geometry>
-                <mesh filename="~/tribot/src/warehouse_robot_sim/meshes/TriOrb300P100_Casters_BlockC_Pall.stl" scale="0.001 0.001 0.001" />
+                <mesh filename="file://$(find warehouse_robot_sim)/meshes/TriOrb300P100_Casters_BlockC_Pall.stl" scale="0.001 0.001 0.001" />
             </geometry>
         </collision>
@@ -573,5 +470,5 @@
             <origin xyz="-0.012 -0.133 0.07" rpy="0.0 0.0 -1.5708" />
             <geometry>
-                <mesh filename="~/tribot/src/warehouse_robot_sim/meshes/TriOrb300P100_PlateA_BLMR5100K-10-B_GPA28GT5150-A-N18.stl" scale="0.001 0.001 0.001" />
+                <mesh filename="file://$(find warehouse_robot_sim)/meshes/TriOrb300P100_PlateA_BLMR5100K-10-B_GPA28GT5150-A-N18.stl" scale="0.001 0.001 0.001" />
             </geometry>
             <material name="white_aluminum">
@@ -582,5 +479,5 @@
             <origin xyz="-0.012 -0.133 0.07" rpy="0.0 0.0 -1.5708" />
             <geometry>
-                <mesh filename="~/tribot/src/warehouse_robot_sim/meshes/TriOrb300P100_PlateA_BLMR5100K-10-B_GPA28GT5150-A-N18.stl" scale="0.001 0.001 0.001" />
+                <mesh filename="file://$(find warehouse_robot_sim)/meshes/TriOrb300P100_PlateA_BLMR5100K-10-B_GPA28GT5150-A-N18.stl" scale="0.001 0.001 0.001" />
             </geometry>
         </collision>
@@ -595,5 +492,5 @@
             <origin xyz="-0.012 -0.123 0.07" rpy="-1.5708 0.0 -1.5708" />
             <geometry>
-                <mesh filename="~/tribot/src/warehouse_robot_sim/meshes/TriOrb300P100_PlateA_BLMR5100K-10-B_Motor.stl" scale="0.001 0.001 0.001" />
+                <mesh filename="file://$(find warehouse_robot_sim)/meshes/TriOrb300P100_PlateA_BLMR5100K-10-B_Motor.stl" scale="0.001 0.001 0.001" />
             </geometry>
             <material name="light_gray">
@@ -604,5 +501,5 @@
             <origin xyz="-0.012 -0.123 0.07" rpy="-1.5708 0.0 -1.5708" />
             <geometry>
-                <mesh filename="~/tribot/src/warehouse_robot_sim/meshes/TriOrb300P100_PlateA_BLMR5100K-10-B_Motor.stl" scale="0.001 0.001 0.001" />
+                <mesh filename="file://$(find warehouse_robot_sim)/meshes/TriOrb300P100_PlateA_BLMR5100K-10-B_Motor.stl" scale="0.001 0.001 0.001" />
             </geometry>
         </collision>
@@ -617,5 +514,5 @@
             <origin xyz="0.123 0.057 0.067" rpy="0.0 0.0 0.523599" />
             <geometry>
-                <mesh filename="~/tribot/src/warehouse_robot_sim/meshes/TriOrb300P100_PlateA_BLMR5100K-10-B_GPA28GT5150-A-N18.stl" scale="0.001 0.001 0.001" />
+                <mesh filename="file://$(find warehouse_robot_sim)/meshes/TriOrb300P100_PlateA_BLMR5100K-10-B_GPA28GT5150-A-N18.stl" scale="0.001 0.001 0.001" />
             </geometry>
             <material name="white_aluminum">
@@ -626,5 +523,5 @@
             <origin xyz="0.123 0.057 0.067" rpy="0.0 0.0 0.523599" />
             <geometry>
-                <mesh filename="~/tribot/src/warehouse_robot_sim/meshes/TriOrb300P100_PlateA_BLMR5100K-10-B_GPA28GT5150-A-N18.stl" scale="0.001 0.001 0.001" />
+                <mesh filename="file://$(find warehouse_robot_sim)/meshes/TriOrb300P100_PlateA_BLMR5100K-10-B_GPA28GT5150-A-N18.stl" scale="0.001 0.001 0.001" />
             </geometry>
         </collision>
@@ -639,5 +536,5 @@
             <origin xyz="0.115 0.052 0.067" rpy="-1.5708 0.0 0.523599" />
             <geometry>
-                <mesh filename="~/tribot/src/warehouse_robot_sim/meshes/TriOrb300P100_PlateA_BLMR5100K-10-B_Motor.stl" scale="0.001 0.001 0.001" />
+                <mesh filename="file://$(find warehouse_robot_sim)/meshes/TriOrb300P100_PlateA_BLMR5100K-10-B_Motor.stl" scale="0.001 0.001 0.001" />
             </geometry>
             <material name="light_gray">
@@ -648,5 +545,5 @@
             <origin xyz="0.115 0.052 0.067" rpy="-1.5708 0.0 0.523599" />
             <geometry>
-                <mesh filename="~/tribot/src/warehouse_robot_sim/meshes/TriOrb300P100_PlateA_BLMR5100K-10-B_Motor.stl" scale="0.001 0.001 0.001" />
+                <mesh filename="file://$(find warehouse_robot_sim)/meshes/TriOrb300P100_PlateA_BLMR5100K-10-B_Motor.stl" scale="0.001 0.001 0.001" />
             </geometry>
         </collision>
@@ -661,5 +558,5 @@
             <origin xyz="-0.111 0.078 0.067" rpy="0.0 0.0 2.61799" />
             <geometry>
-                <mesh filename="~/tribot/src/warehouse_robot_sim/meshes/TriOrb300P100_PlateA_BLMR5100K-10-B_GPA28GT5150-A-N18.stl" scale="0.001 0.001 0.001" />
+                <mesh filename="file://$(find warehouse_robot_sim)/meshes/TriOrb300P100_PlateA_BLMR5100K-10-B_GPA28GT5150-A-N18.stl" scale="0.001 0.001 0.001" />
             </geometry>
             <material name="white_aluminum">
@@ -670,5 +567,5 @@
             <origin xyz="-0.111 0.078 0.067" rpy="0.0 0.0 2.61799" />
             <geometry>
-                <mesh filename="~/tribot/src/warehouse_robot_sim/meshes/TriOrb300P100_PlateA_BLMR5100K-10-B_GPA28GT5150-A-N18.stl" scale="0.001 0.001 0.001" />
+                <mesh filename="file://$(find warehouse_robot_sim)/meshes/TriOrb300P100_PlateA_BLMR5100K-10-B_GPA28GT5150-A-N18.stl" scale="0.001 0.001 0.001" />
             </geometry>
         </collision>
@@ -683,5 +580,5 @@
             <origin xyz="-0.103 0.073 0.067" rpy="-1.5708 0.0 2.61799" />
             <geometry>
-                <mesh filename="~/tribot/src/warehouse_robot_sim/meshes/TriOrb300P100_PlateA_BLMR5100K-10-B_Motor.stl" scale="0.001 0.001 0.001" />
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