Commit message: Removed config error

File: warehouse_robot_sim/urdf/oakd.urdf.xacro (robot description, xacro)
@@ -1,180 +1,90 @@
-<?xml version="1.0" ?>
-<!--  xacro macros for oakd mount -->
-<robot name="oakd" xmlns:xacro="http://ros.org/wiki/xacro">
-      <xacro:macro name="oakd_link" params="mount_point">
-      <xacro:property name="oakd_length" value="0.0803" />
-      <xacro:property name="oakd_width" value="0.0957" />
-      <xacro:property name="oakd_depth" value="0.1267" />
-      <xacro:property name="oakd_mass" value="0.15" />
-      <link name="oakd_${mount_point}">
-             <pose>0.0 0.0 0.0 0.0 0.0 0.0</pose>
-          <visual>
-              <origin rpy="0 0 0" xyz="0 0 0" />
-              <geometry>
-                      <mesh filename="../meshes/sensors/OAK-D.dae" />
-              </geometry>
-               <material name="black" />
-          </visual>
-          <collision>
-              <origin rpy="0 0 0" xyz="0 0 0" />
-              <geometry>
-                  <box size="${oakd_length} ${oakd_width} ${oakd_depth}"/>
-              </geometry>
-          </collision>
-          <xacro:solid_cuboid_inertial
-              rpy="0 0 0" xyz="0 0 0"
-              mass="${oakd_mass}"
-              x="${oakd_length}" y="${oakd_width}" z="${oakd_depth}" />
-      </link>
-      <!-- Add dummy joint for camera_optical_frame to link back to base_link -->
-      <joint name="camera_optical_joint" type="fixed">
-      <!-- Point cloud frustrum is 90 degrees off from visual frame -->
-           <origin rpy="-1.57079632769 0 -1.570796332769" xyz="0 0 0" />
-	   <parent link="oakd_${mount_point}" />
-	   <child link="camera_optical_frame" />
-	</joint>
-	<!-- Add dummy link for camera_optical_frame to link back to base_link -->
-        <link name="camera_optical_frame">
-        <inertial>
-	  <mass value="0.001" />
-	  <origin xyz="0 0 0" />
-	  <inertia ixx="0.0001" ixy="0.0" ixz="0.0" iyy="0.0001" iyz="0.0" izz="0.0001" />
-          </inertial>
-  </link>
-  <!-- Dummy joints for rgb camera to link back to base_link -->
-        <joint name="camera_rgb_optical_joint" type="fixed">
-           <origin rpy="0 0 0" xyz="0 0 0" />
-	   <parent link="oakd_${mount_point}" />
-	   <child link="camera_rgb_optical_frame" />
-	</joint>
-	<!-- Add dummy link for camera_optical_frame to link back to base_link -->
-        <link name="camera_rgb_optical_frame">
-        <inertial>
-	  <mass value="0.001" />
-	  <origin xyz="0 0 0" />
-	  <inertia ixx="0.0001" ixy="0.0" ixz="0.0" iyy="0.0001" iyz="0.0" izz="0.0001" />
-          </inertial>
-  </link>
-  <!-- Gazebo plugin for greyscale left/right stereo pairs -->
-      <gazebo reference="oakd_${mount_point}">
-    <material>Gazebo/DarkGrey</material>
-    <sensor type="multicamera" name="stereo_camera">
-      <update_rate>30.0</update_rate>
-      <camera name="left">
-        <horizontal_fov>1.2566</horizontal_fov>
-        <image>
-          <width>1200</width>
-          <height>800</height>
-	  <format>L8</format>
-	  <!--   <format>R8G8B8</format> -->
-        </image>
-        <clip>
-          <near>0.3</near>
-          <far>35</far>
-        </clip>
-        <noise>
-          <type>gaussian</type>
-          <mean>0.0</mean>
-          <stddev>0.007</stddev>
-        </noise>
-      </camera>
-      <camera name="right">
-        <pose>0 -0.07 0 0 0 0</pose>
-        <horizontal_fov>1.1.2566</horizontal_fov>
-        <image>
-          <width>1200</width>
-          <height>800</height>
-	  <format>L8</format>
-	  <!--   <format>R8G8B8</format> -->
-        </image>
-        <clip>
-          <near>0.3</near>
-          <far>35</far>
-        </clip>
-        <noise>
-          <type>gaussian</type>
-          <mean>0.0</mean>
-          <stddev>0.007</stddev>
-        </noise>
-      </camera>
-      <plugin name="stereo_camera_controller" filename="libgazebo_ros_multicamera.so">
-        <alwaysOn>true</alwaysOn>
-        <updateRate>0.0</updateRate>
-	<cameraName>oakd_${mount_point}/camera</cameraName>
-        <imageTopicName>image_raw</imageTopicName>
-        <cameraInfoTopicName>camera_info</cameraInfoTopicName>
-	<frameName>camera_optical_frame</frameName>
-        <!--<rightFrameName>right_camera_optical_frame</rightFrameName>-->
-        <hackBaseline>0.075</hackBaseline>
-        <distortionK1>0.0</distortionK1>
-        <distortionK2>0.0</distortionK2>
-        <distortionK3>0.0</distortionK3>
-        <distortionT1>0.0</distortionT1>
-        <distortionT2>0.0</distortionT2>
-      </plugin>
-    </sensor>
-  </gazebo>
- <!-- Gazebo plugin for center RGB camera -->
-   <gazebo reference="oakd_${mount_point}">
-      <material>Gazebo/White</material>
-      <sensor type="camera" name="oakd_rgb_${mount_point}">
-      <update_rate>30.0</update_rate>
-      <camera name="head">
-        <horizontal_fov>1.3962634</horizontal_fov>
-        <image>
-          <width>800</width>
-          <height>800</height>
-          <format>R8G8B8</format>
-        </image>
-        <clip>
-          <near>0.02</near>
-          <far>300</far>
-        </clip>
-        <noise>
-          <type>gaussian</type>
-          <!-- Noise is sampled independently per pixel on each frame.
-               That pixel's noise value is added to each of its color
-               channels, which at that point lie in the range [0,1]. -->
-          <mean>0.0</mean>
-          <stddev>0.007</stddev>
-        </noise>
-      </camera>
-      <plugin name="camera_controller" filename="libgazebo_ros_camera.so">
-        <alwaysOn>true</alwaysOn>
-        <updateRate>0.0</updateRate>
-        <cameraName>oakd_rgb_${mount_point}</cameraName>
-        <imageTopicName>image_raw</imageTopicName>
-        <cameraInfoTopicName>camera_info</cameraInfoTopicName>
-        <frameName>camera_rgb_link_optical</frameName>
-        <!-- setting hackBaseline to anything but 0.0 will cause a misalignment
-            between the gazebo sensor image and the frame it is supposed to
-            be attached to -->
-        <hackBaseline>0.0</hackBaseline>
-        <distortionK1>0.0</distortionK1>
-        <distortionK2>0.0</distortionK2>
-        <distortionK3>0.0</distortionK3>
-        <distortionT1>0.0</distortionT1>
-        <distortionT2>0.0</distortionT2>
-        <CxPrime>0</CxPrime>
-        <Cx>0.0</Cx>
-        <Cy>0.0</Cy>
-        <focalLength>0.0</focalLength>
-      </plugin>
-    </sensor>
-  </gazebo>
-      <gazebo reference="oakd_joint_${mount_point}">
-          <!-- <disableFixedJointLumping>true</disableFixedJointLumping>  -->
-          <!-- <preserveFixedJoint>true</preserveFixedJoint> -->
-      </gazebo>
-    </xacro:macro>
-    <xacro:macro name="oakd_joint" params="x y z roll pitch yaw mount_point" >
-        <joint name="oakd_joint_${mount_point}" type="fixed">
-                <origin rpy="${roll} ${pitch} ${yaw}" xyz="${x+0.1} ${y-0.01} ${z}"/>
-            <parent link="base_link" />
-            <child link="oakd_${mount_point}" />
-        </joint>
-        <gazebo reference="oakd_joint_${mount_point}">
-            <preserveFixedJoint>true</preserveFixedJoint>
-        </gazebo>
-    </xacro:macro>
+<robot xmlns:xacro="http://ros.org/wiki/xacro">
+  <xacro:property name="M_PI" value="3.1415926535897931" />
+  <xacro:macro name="depth_sensor" params="*origin">
+    <link name="camera_link">
+      <visual>
+        <origin xyz="0 0 0" rpy="0 0 0"/>
+        <geometry>
+          <box size="0.030 0.124 0.030"/>
+          <!-- <mesh filename="" scale="0.001 0.001 0.001"/> -->
+        </geometry>
+        <material name="red">
+          <color rgba="0.416 0.051 0.047 1.0"/>
+        </material>
+      </visual>
+      <collision>
+        <origin xyz="0 0 0" rpy="0 0 0"/>
+        <geometry>
+          <box size="0.030 0.124 0.030"/>
+        </geometry>
+      </collision>
+      <inertial>
+        <origin xyz="0 0 0" rpy="0 0 0"/>
+        <mass value="0.135"/>
+        <inertia ixx="${(1/12) * 0.135 * ((0.124  * 0.124)  + (0.030 * 0.030))}" ixy="0.0" ixz="0.0"
+                 iyy="${(1/12) * 0.135 * ((0.030 * 0.030) + (0.030 * 0.030))}" iyz="0.0"
+                 izz="${(1/12) * 0.135 * ((0.030 * 0.030) + (0.124  * 0.124))}"/>
+      </inertial>
+    </link>
+    <gazebo reference="camera_link">
+      <visual>
+        <material>
+          <ambient>0.416 0.051 0.047 1.0</ambient>
+          <diffuse>0.416 0.051 0.047 1.0</diffuse>
+          <specular>0.416 0.051 0.047 1.0</specular>
+          <emissive>0.416 0.051 0.047 1.0</emissive>
+        </material>
+      </visual>
+    </gazebo>rgb(213,28,40)
+    <joint name="camera_to_base_link" type="fixed">
+      <parent link="base_link"/>
+      <child link="camera_link"/>
+      <xacro:insert_block name="origin" />
+    </joint>
+    <link name="camera_depth_link"/>
+    <joint name="camera_depth_joint" type="fixed">
+      <origin xyz="0 0 0" rpy="-1.57 0 -1.57"/>
+      <parent link="camera_link"/>
+      <child link="camera_depth_link"/>
+    </joint>
+    <!-- https://github.com/ros-simulation/gazebo_ros_pkgs/wiki/ROS-2-Migration:-Camera#gazebo_ros_camera -->
+    <gazebo reference="camera_link">
+      <sensor name="camera" type="depth">
+        <always_on>true</always_on>
+        <update_rate>30.0</update_rate>
+        <camera name="camera">
+          <horizontal_fov>1.50098</horizontal_fov>
+          <image>
+            <width>640</width>
+            <height>480</height>
+            <format>R8G8B8</format>
+          </image>
+        </camera>
+        <plugin name="camera_controller" filename="libgazebo_ros_camera.so">
+          <ros>
+            <remapping>/camera/camera_info:=/camera/color/camera_info</remapping>
+            <remapping>/camera/image_raw:=/camera/color/image_raw</remapping>
+            <remapping>/camera/points:=/camera/depth/color/points</remapping>
+            <remapping>/camera/depth/image_raw:=/camera/depth/image_rect_raw</remapping>
+            <qos>
+              <topic name="/camera/depth/color/points">
+                <publisher>
+                  <reliability>best_effort</reliability>
+                </publisher>
+              </topic>
+            </qos>
+          </ros>
+          <min_depth>0.015</min_depth>
+          <max_depth>3.0</max_depth>
+          <hack_baseline>0.07</hack_baseline>
+          <frame_name>camera_depth_link</frame_name>
+          <distortion_k1>0.00000001</distortion_k1>
+          <distortion_k2>0.00000001</distortion_k2>
+          <distortion_k3>0.00000001</distortion_k3>
+          <distortion_t1>0.00000001</distortion_t1>
+          <distortion_t2>0.00000001</distortion_t2>
+        </plugin>
+      </sensor>
+    </gazebo>
+  </xacro:macro>
 </robot>

Commit message: nav2 working

File: warehouse_robot_sim/urdf/TriBot_Oakd.urdf.xacro (robot description, xacro)
@@ -3,7 +3,7 @@
   <xacro:include filename="$(find warehouse_robot_sim)/urdf/oakd.urdf.xacro"/>
   <xacro:include filename="$(find warehouse_robot_sim)/urdf/omni_controller.urdf.xacro" />
-<link name="base_footprint">
+<link name="base_link">
 </link>
-  <link name="base_link">
+  <link name="robot_base">
     <inertial>
       <origin xyz="0 0 0" rpy="0 0 0"/>
@@ -28,7 +28,7 @@
   </link>
 <joint name="base_joint" type="fixed">
-    <origin xyz="0.0 0.0 0.15" rpy="0.0 0.0 1.57"/>
-    <parent link="base_footprint"/>
-    <child link="base_link"/>
+    <origin xyz="0.0 0.0 0.0" rpy="0.0 0.0 1.57"/>
+    <parent link="base_link"/>
+    <child link="robot_base"/>
  </joint>
   <link name="TriOrb300P100_TopPlate">
@@ -55,5 +55,5 @@
   </link>
   <joint name="TriOrb300P100_TopPlate_joint" type="fixed">
-    <parent link="base_link"/>
+    <parent link="robot_base"/>
     <child link="TriOrb300P100_TopPlate"/>
     <origin xyz="0 0 0" rpy="0 0 0"/>
@@ -82,5 +82,5 @@
   </link>
   <joint name="TriOrb300P100_Ball100_1_joint" type="fixed">
-    <parent link="base_link"/>
+    <parent link="robot_base"/>
     <child link="TriOrb300P100_Ball100_1"/>
     <origin xyz="0 0 0" rpy="0 0 0"/>
@@ -131,10 +131,10 @@
   </link>
   <joint name="TriOrb300P100_Ball100_2_joint" type="fixed">
-    <parent link="base_link"/>
+    <parent link="robot_base"/>
     <child link="TriOrb300P100_Ball100_2"/>
     <origin xyz="0 0 0" rpy="0 0 0"/>
   </joint>
   <joint name="TriOrb300P100_Ball100_3_joint" type="fixed">
-    <parent link="base_link"/>
+    <parent link="robot_base"/>
     <child link="TriOrb300P100_Ball100_3"/>
     <origin xyz="0 0 0" rpy="0 0 0"/>
@@ -162,5 +162,5 @@
   </link>
   <joint name="TriOrb300P100_PlateA_PlateA-1_joint" type="fixed">
-    <parent link="base_link"/>
+    <parent link="robot_base"/>
     <child link="TriOrb300P100_PlateA_PlateA-1"/>
     <origin xyz="0 0 0" rpy="0 0 0"/>
@@ -209,10 +209,10 @@
   </link>
   <joint name="TriOrb300P100_PlateA_PlateA-2_joint" type="fixed">
-    <parent link="base_link"/>
+    <parent link="robot_base"/>
     <child link="TriOrb300P100_PlateA_PlateA-2"/>
     <origin xyz="0 0 0" rpy="0 0 0"/>
   </joint>
   <joint name="TriOrb300P100_PlateA_PlateA-3_joint" type="fixed">
-    <parent link="base_link"/>
+    <parent link="robot_base"/>
     <child link="TriOrb300P100_PlateA_PlateA-3"/>
     <origin xyz="0 0 0" rpy="0 0 0"/>
@@ -285,15 +285,15 @@
   </link>
   <joint name="TriOrb300P100_Casters_BlockC_BlockC1_joint" type="fixed">
-    <parent link="base_link"/>
+    <parent link="robot_base"/>
     <child link="TriOrb300P100_Casters_BlockC_BlockC1"/>
     <origin xyz="0 0 0" rpy="0 0 0"/>
   </joint>
   <joint name="TriOrb300P100_Casters_BlockC_BlockC2_joint" type="fixed">
-    <parent link="base_link"/>
+    <parent link="robot_base"/>
     <child link="TriOrb300P100_Casters_BlockC_BlockC2"/>
     <origin xyz="0 0 0" rpy="0 0 0"/>
   </joint>
   <joint name="TriOrb300P100_Casters_BlockC_BlockC3_joint" type="fixed">
-    <parent link="base_link"/>
+    <parent link="robot_base"/>
     <child link="TriOrb300P100_Casters_BlockC_BlockC3"/>
     <origin xyz="0 0 0" rpy="0 0 0"/>
@@ -432,30 +432,30 @@
   </link>
   <joint name="TriOrb300P100_Casters_BlockC_Pall1a_joint" type="fixed">
-    <parent link="base_link"/>
+    <parent link="robot_base"/>
     <child link="TriOrb300P100_Casters_BlockC_Pall1a"/>
     <origin xyz="0 0 0" rpy="0 0 0"/>
   </joint>
   <joint name="TriOrb300P100_Casters_BlockC_Pall1b_joint" type="fixed">
-    <parent link="base_link"/>
+    <parent link="robot_base"/>
     <child link="TriOrb300P100_Casters_BlockC_Pall1b"/>
     <origin xyz="0 0 0" rpy="0 0 0"/>
   </joint>
   <joint name="TriOrb300P100_Casters_BlockC_Pall2a_joint" type="fixed">
-    <parent link="base_link"/>
+    <parent link="robot_base"/>
     <child link="TriOrb300P100_Casters_BlockC_Pall2a"/>
     <origin xyz="0 0 0" rpy="0 0 0"/>
   </joint>
   <joint name="TriOrb300P100_Casters_BlockC_Pall2b_joint" type="fixed">
-    <parent link="base_link"/>
+    <parent link="robot_base"/>
     <child link="TriOrb300P100_Casters_BlockC_Pall2b"/>
     <origin xyz="0 0 0" rpy="0 0 0"/>
   </joint>
   <joint name="TriOrb300P100_Casters_BlockC_Pall3a_joint" type="fixed">
-    <parent link="base_link"/>
+    <parent link="robot_base"/>
     <child link="TriOrb300P100_Casters_BlockC_Pall3a"/>
     <origin xyz="0 0 0" rpy="0 0 0"/>
   </joint>
   <joint name="TriOrb300P100_Casters_BlockC_Pall3b_joint" type="fixed">
-    <parent link="base_link"/>
+    <parent link="robot_base"/>
     <child link="TriOrb300P100_Casters_BlockC_Pall3b"/>
     <origin xyz="0 0 0" rpy="0 0 0"/>
@@ -594,30 +594,30 @@
   </link>
   <joint name="TriOrb300P100_PlateA1_BLMR5100K-10-B_GPA28GT5150-A-N18_joint" type="fixed">
-    <parent link="base_link"/>
+    <parent link="robot_base"/>
     <child link="TriOrb300P100_PlateA1_BLMR5100K-10-B_GPA28GT5150-A-N18"/>
     <origin xyz="0 0 0" rpy="0 0 0"/>
   </joint>
   <joint name="TriOrb300P100_PlateA1_BLMR5100K-10-B_Motor_joint" type="fixed">
-    <parent link="base_link"/>
+    <parent link="robot_base"/>
     <child link="TriOrb300P100_PlateA1_BLMR5100K-10-B_Motor"/>
     <origin xyz="0 0 0" rpy="0 0 0"/>
   </joint>
   <joint name="TriOrb300P100_PlateA2_BLMR5100K-10-B_GPA28GT5150-A-N18_joint" type="fixed">
-    <parent link="base_link"/>
+    <parent link="robot_base"/>
     <child link="TriOrb300P100_PlateA2_BLMR5100K-10-B_GPA28GT5150-A-N18"/>
     <origin xyz="0 0 0" rpy="0 0 0"/>
   </joint>
   <joint name="TriOrb300P100_PlateA2_BLMR5100K-10-B_Motor_joint" type="fixed">
-    <parent link="base_link"/>
+    <parent link="robot_base"/>
     <child link="TriOrb300P100_PlateA2_BLMR5100K-10-B_Motor"/>
     <origin xyz="0 0 0" rpy="0 0 0"/>
   </joint>
   <joint name="TriOrb300P100_PlateA3_BLMR5100K-10-B_GPA28GT5150-A-N18_joint" type="fixed">
-    <parent link="base_link"/>
+    <parent link="robot_base"/>
     <child link="TriOrb300P100_PlateA3_BLMR5100K-10-B_GPA28GT5150-A-N18"/>
     <origin xyz="0 0 0" rpy="0 0 0"/>
   </joint>
   <joint name="TriOrb300P100_PlateA3_BLMR5100K-10-B_Motor_joint" type="fixed">
-    <parent link="base_link"/>
+    <parent link="robot_base"/>
     <child link="TriOrb300P100_PlateA3_BLMR5100K-10-B_Motor"/>
     <origin xyz="0 0 0" rpy="0 0 0"/>
@@ -690,15 +690,15 @@
   </link>
   <joint name="TriOrb300P100_PlateA1_Belt_joint" type="fixed">
-    <parent link="base_link"/>
+    <parent link="robot_base"/>
     <child link="TriOrb300P100_PlateA1_Belt"/>
     <origin xyz="0 0 0" rpy="0 0 0"/>
   </joint>
   <joint name="TriOrb300P100_PlateA2_Belt_joint" type="fixed">
-    <parent link="base_link"/>
+    <parent link="robot_base"/>
     <child link="TriOrb300P100_PlateA2_Belt"/>
     <origin xyz="0 0 0" rpy="0 0 0"/>
   </joint>
   <joint name="TriOrb300P100_PlateA3_Belt_joint" type="fixed">
-    <parent link="base_link"/>
+    <parent link="robot_base"/>
     <child link="TriOrb300P100_PlateA3_Belt"/>
     <origin xyz="0 0 0" rpy="0 0 0"/>
@@ -837,30 +837,30 @@
   </link>
   <joint name="TriOrb300P100_PlateA1_Axis1_GPA25GT5150-A-N15_joint" type="fixed">
-    <parent link="base_link"/>
+    <parent link="robot_base"/>
     <child link="TriOrb300P100_PlateA1_Axis1_GPA25GT5150-A-N15"/>
     <origin xyz="0 0 0" rpy="0 0 0"/>
   </joint>
   <joint name="TriOrb300P100_PlateA1_Axis2_GPA25GT5150-A-N15_joint" type="fixed">
-    <parent link="base_link"/>
+    <parent link="robot_base"/>
     <child link="TriOrb300P100_PlateA1_Axis2_GPA25GT5150-A-N15"/>
     <origin xyz="0 0 0" rpy="0 0 0"/>
   </joint>
   <joint name="TriOrb300P100_PlateA2_Axis1_GPA25GT5150-A-N15_joint" type="fixed">
-    <parent link="base_link"/>
+    <parent link="robot_base"/>
     <child link="TriOrb300P100_PlateA2_Axis1_GPA25GT5150-A-N15"/>
     <origin xyz="0 0 0" rpy="0 0 0"/>
   </joint>
   <joint name="TriOrb300P100_PlateA2_Axis2_GPA25GT5150-A-N15_joint" type="fixed">
-    <parent link="base_link"/>
+    <parent link="robot_base"/>
     <child link="TriOrb300P100_PlateA2_Axis2_GPA25GT5150-A-N15"/>
     <origin xyz="0 0 0" rpy="0 0 0"/>
   </joint>
   <joint name="TriOrb300P100_PlateA3_Axis1_GPA25GT5150-A-N15_joint" type="fixed">
-    <parent link="base_link"/>
+    <parent link="robot_base"/>
     <child link="TriOrb300P100_PlateA3_Axis1_GPA25GT5150-A-N15"/>
     <origin xyz="0 0 0" rpy="0 0 0"/>
   </joint>
   <joint name="TriOrb300P100_PlateA3_Axis2_GPA25GT5150-A-N15_joint" type="fixed">
-    <parent link="base_link"/>
+    <parent link="robot_base"/>
     <child link="TriOrb300P100_PlateA3_Axis2_GPA25GT5150-A-N15"/>
     <origin xyz="0 0 0" rpy="0 0 0"/>
@@ -999,30 +999,30 @@
   </link>
   <joint name="TriOrb300P100_PlateA1_Idlar1_AFBD15-30_joint" type="fixed">
-    <parent link="base_link"/>
+    <parent link="robot_base"/>
     <child link="TriOrb300P100_PlateA1_Idlar1_AFBD15-30"/>
     <origin xyz="0 0 0" rpy="0 0 0"/>
   </joint>
   <joint name="TriOrb300P100_PlateA1_Idlar2_AFBD15-30_joint" type="fixed">
-    <parent link="base_link"/>
+    <parent link="robot_base"/>
     <child link="TriOrb300P100_PlateA1_Idlar2_AFBD15-30"/>
     <origin xyz="0 0 0" rpy="0 0 0"/>
   </joint>
   <joint name="TriOrb300P100_PlateA2_Idlar1_AFBD15-30_joint" type="fixed">
-    <parent link="base_link"/>
+    <parent link="robot_base"/>
     <child link="TriOrb300P100_PlateA2_Idlar1_AFBD15-30"/>
     <origin xyz="0 0 0" rpy="0 0 0"/>
   </joint>
   <joint name="TriOrb300P100_PlateA2_Idlar2_AFBD15-30_joint" type="fixed">
-    <parent link="base_link"/>
+    <parent link="robot_base"/>
     <child link="TriOrb300P100_PlateA2_Idlar2_AFBD15-30"/>
     <origin xyz="0 0 0" rpy="0 0 0"/>
   </joint>
   <joint name="TriOrb300P100_PlateA3_Idlar1_AFBD15-30_joint" type="fixed">
-    <parent link="base_link"/>
+    <parent link="robot_base"/>
     <child link="TriOrb300P100_PlateA3_Idlar1_AFBD15-30"/>
     <origin xyz="0 0 0" rpy="0 0 0"/>
   </joint>
   <joint name="TriOrb300P100_PlateA3_Idlar2_AFBD15-30_joint" type="fixed">
-    <parent link="base_link"/>
+    <parent link="robot_base"/>
     <child link="TriOrb300P100_PlateA3_Idlar2_AFBD15-30"/>
     <origin xyz="0 0 0" rpy="0 0 0"/>
@@ -1051,5 +1051,5 @@
   </link>
   <joint name="TriOrb300P100_UnderPlate_joint" type="fixed">
-    <parent link="base_link"/>
+    <parent link="robot_base"/>
     <child link="TriOrb300P100_UnderPlate"/>
     <origin xyz="0 0 0" rpy="0 0 0"/>

File: warehouse_robot_sim/urdf/oakd.urdf.xacro (robot description, xacro)
@@ -37,6 +37,6 @@
       </visual>
     </gazebo>rgb(213,28,40)
-    <joint name="camera_to_base_link" type="fixed">
-      <parent link="base_link"/>
+    <joint name="camera_to_base" type="fixed">
+      <parent link="robot_base"/>
       <child link="camera_link"/>
       <xacro:insert_block name="origin" />

File: warehouse_robot_sim/urdf/omni_controller.urdf.xacro (robot description, xacro)
@@ -10,5 +10,5 @@
       <odometry_frame>odom</odometry_frame>
       <odometry_rate>20.0</odometry_rate>
-      <robot_base_frame>base_footprint</robot_base_frame>
+      <robot_base_frame>base_link</robot_base_frame>
       <publish_odom>true</publish_odom>
       <publish_odom_tf>true</publish_odom_tf>
