Commit message: Initial push on adam_simulation branch

File: triorb_descriptions/urdf/guider.urdf.copy.xacro (robot description, xacro)
@@ -1,8 +1,5 @@
 <?xml version="1.0" ?>
 <robot name="TriOrb300P100" xmlns:xacro="http://ros.org/wiki/xacro">
-  <xacro:include filename="$(find warehouse_robot_sim)/urdf/oakd.urdf.xacro"/>
-  <xacro:include filename="$(find warehouse_robot_sim)/urdf/omni_controller.urdf.xacro" />
-<link name="base_link">
-</link>
+<link name="base_link"/>
   <link name="robot_base">
     <inertial>
@@ -14,5 +11,5 @@
         <origin xyz="0.0 0.0 0.0" rpy="0.0 0.0 0.0" />
         <geometry>
-            <mesh filename="file://$(find warehouse_robot_sim)/meshes/TriOrb300P100_UnderPlate.stl" scale="0.001 0.001 0.001" />
+            <mesh filename="file://$(find triorb_descriptions)/meshes/TriOrb300P100_UnderPlate.stl" scale="0.001 0.001 0.001" />
         </geometry>
         <material name="sus">
@@ -23,13 +20,13 @@
         <origin xyz="0.0 0.0 0.0" rpy="0.0 0.0 0.0" />
         <geometry>
-            <mesh filename="file://$(find warehouse_robot_sim)/meshes/TriOrb300P100_UnderPlate.stl" scale="0.001 0.001 0.001" />
+            <mesh filename="file://$(find triorb_descriptions)/meshes/TriOrb300P100_UnderPlate.stl" scale="0.001 0.001 0.001" />
         </geometry>
     </collision>
   </link>
-<joint name="base_joint" type="fixed">
-    <origin xyz="0.0 0.0 0.0" rpy="0.0 0.0 1.57"/>
+    <joint name="base_joint" type="fixed">
     <parent link="base_link"/>
     <child link="robot_base"/>
- </joint>
+    <origin xyz="0 0 0" rpy="0 0 1.57"/>
+  </joint>
   <link name="TriOrb300P100_TopPlate">
     <inertial>
@@ -41,5 +38,5 @@
         <origin xyz="0.0 0.0 0.0" rpy="0.0 -0.0 0.0" />
         <geometry>
-            <mesh filename="file://$(find warehouse_robot_sim)/meshes/TriOrb300P100_TopPlate.stl" scale="0.001 0.001 0.001" />
+            <mesh filename="file://$(find triorb_descriptions)/meshes/TriOrb300P100_TopPlate.stl" scale="0.001 0.001 0.001" />
         </geometry>
         <material name="dark_gray">
@@ -50,5 +47,5 @@
         <origin xyz="0.0 0.0 0.0" rpy="0.0 -0.0 0.0" />
         <geometry>
-            <mesh filename="file://$(find warehouse_robot_sim)/meshes/TriOrb300P100_TopPlate.stl" scale="0.001 0.001 0.001" />
+            <mesh filename="file://$(find triorb_descriptions)/meshes/TriOrb300P100_TopPlate.stl" scale="0.001 0.001 0.001" />
         </geometry>
     </collision>
@@ -148,5 +145,5 @@
         <origin xyz="0.0 -0.131 0.064" rpy="1.5708 0.0 0.0" />
         <geometry>
-            <mesh filename="file://$(find warehouse_robot_sim)/meshes/TriOrb300P100_PlateA_PlateA-1.stl" scale="0.001 0.001 0.001" />
+            <mesh filename="file://$(find triorb_descriptions)/meshes/TriOrb300P100_PlateA_PlateA-1.stl" scale="0.001 0.001 0.001" />
         </geometry>
         <material name="aluminum">
@@ -157,5 +154,5 @@
         <origin xyz="0.0 -0.131 0.064" rpy="1.5708 0.0 0.0" />
         <geometry>
-            <mesh filename="file://$(find warehouse_robot_sim)/meshes/TriOrb300P100_PlateA_PlateA-1.stl" scale="0.001 0.001 0.001" />
+            <mesh filename="file://$(find triorb_descriptions)/meshes/TriOrb300P100_PlateA_PlateA-1.stl" scale="0.001 0.001 0.001" />
         </geometry>
     </collision>
@@ -174,5 +171,5 @@
         <origin xyz="0.115 0.067 0.064" rpy="1.5708 0.0 2.0944" />
         <geometry>
-            <mesh filename="file://$(find warehouse_robot_sim)/meshes/TriOrb300P100_PlateA_PlateA-1.stl" scale="0.001 0.001 0.001" />
+            <mesh filename="file://$(find triorb_descriptions)/meshes/TriOrb300P100_PlateA_PlateA-1.stl" scale="0.001 0.001 0.001" />
         </geometry>
         <material name="aluminum">
@@ -183,5 +180,5 @@
         <origin xyz="0.115 0.067 0.064" rpy="1.5708 0.0 2.0944" />
         <geometry>
-            <mesh filename="file://$(find warehouse_robot_sim)/meshes/TriOrb300P100_PlateA_PlateA-1.stl" scale="0.001 0.001 0.001" />
+            <mesh filename="file://$(find triorb_descriptions)/meshes/TriOrb300P100_PlateA_PlateA-1.stl" scale="0.001 0.001 0.001" />
         </geometry>
     </collision>
@@ -195,5 +192,5 @@
         <origin xyz="-0.115 0.067 0.064" rpy="1.5708 0.0 -2.0944" />
         <geometry>
-            <mesh filename="file://$(find warehouse_robot_sim)/meshes/TriOrb300P100_PlateA_PlateA-1.stl" scale="0.001 0.001 0.001" />
+            <mesh filename="file://$(find triorb_descriptions)/meshes/TriOrb300P100_PlateA_PlateA-1.stl" scale="0.001 0.001 0.001" />
         </geometry>
         <material name="aluminum">
@@ -204,5 +201,5 @@
         <origin xyz="-0.115 0.067 0.064" rpy="1.5708 0.0 -2.0944" />
         <geometry>
-            <mesh filename="file://$(find warehouse_robot_sim)/meshes/TriOrb300P100_PlateA_PlateA-1.stl" scale="0.001 0.001 0.001" />
+            <mesh filename="file://$(find triorb_descriptions)/meshes/TriOrb300P100_PlateA_PlateA-1.stl" scale="0.001 0.001 0.001" />
         </geometry>
     </collision>
@@ -227,5 +224,5 @@
             <origin xyz="0.0 0.226 0.138" rpy="0.0 3.1415 -1.5708" />
             <geometry>
-                <mesh filename="file://$(find warehouse_robot_sim)/meshes/TriOrb300P100_Casters_BlockC_BlockC1.stl" scale="0.001 0.001 0.001" />
+                <mesh filename="file://$(find triorb_descriptions)/meshes/TriOrb300P100_Casters_BlockC_BlockC1.stl" scale="0.001 0.001 0.001" />
             </geometry>
             <material name="dark_gray">
@@ -236,5 +233,5 @@
             <origin xyz="0.0 0.226 0.138" rpy="0.0 3.1415 -1.5708" />
             <geometry>
-                <mesh filename="file://$(find warehouse_robot_sim)/meshes/TriOrb300P100_Casters_BlockC_BlockC1.stl" scale="0.001 0.001 0.001" />
+                <mesh filename="file://$(find triorb_descriptions)/meshes/TriOrb300P100_Casters_BlockC_BlockC1.stl" scale="0.001 0.001 0.001" />
             </geometry>
         </collision>
@@ -249,5 +246,5 @@
             <origin xyz="-0.196 -0.113 0.138" rpy="0.0 3.1415 0.521" />
             <geometry>
-                <mesh filename="file://$(find warehouse_robot_sim)/meshes/TriOrb300P100_Casters_BlockC_BlockC1.stl" scale="0.001 0.001 0.001" />
+                <mesh filename="file://$(find triorb_descriptions)/meshes/TriOrb300P100_Casters_BlockC_BlockC1.stl" scale="0.001 0.001 0.001" />
             </geometry>
             <material name="dark_gray">
@@ -258,5 +255,5 @@
             <origin xyz="-0.196 -0.113 0.138" rpy="0.0 3.1415 0.521" />
             <geometry>
-                <mesh filename="file://$(find warehouse_robot_sim)/meshes/TriOrb300P100_Casters_BlockC_BlockC1.stl" scale="0.001 0.001 0.001" />
+                <mesh filename="file://$(find triorb_descriptions)/meshes/TriOrb300P100_Casters_BlockC_BlockC1.stl" scale="0.001 0.001 0.001" />
             </geometry>
         </collision>
@@ -271,5 +268,5 @@
             <origin xyz="0.196 -0.113 0.138" rpy="0.0 3.1415 2.6154" />
             <geometry>
-                <mesh filename="file://$(find warehouse_robot_sim)/meshes/TriOrb300P100_Casters_BlockC_BlockC1.stl" scale="0.001 0.001 0.001" />
+                <mesh filename="file://$(find triorb_descriptions)/meshes/TriOrb300P100_Casters_BlockC_BlockC1.stl" scale="0.001 0.001 0.001" />
             </geometry>
             <material name="dark_gray">
@@ -280,5 +277,5 @@
             <origin xyz="0.196 -0.113 0.138" rpy="0.0 3.1415 2.6154" />
             <geometry>
-                <mesh filename="file://$(find warehouse_robot_sim)/meshes/TriOrb300P100_Casters_BlockC_BlockC1.stl" scale="0.001 0.001 0.001" />
+                <mesh filename="file://$(find triorb_descriptions)/meshes/TriOrb300P100_Casters_BlockC_BlockC1.stl" scale="0.001 0.001 0.001" />
             </geometry>
         </collision>
@@ -308,5 +305,5 @@
             <origin xyz="-0.057 0.222 0.138" rpy="0 3.1415 2.617901" />
             <geometry>
-                <mesh filename="file://$(find warehouse_robot_sim)/meshes/TriOrb300P100_Casters_BlockC_Pall.stl" scale="0.001 0.001 0.001" />
+                <mesh filename="file://$(find triorb_descriptions)/meshes/TriOrb300P100_Casters_BlockC_Pall.stl" scale="0.001 0.001 0.001" />
             </geometry>
             <material name="dark_gray">
@@ -317,5 +314,5 @@
             <origin xyz="-0.057 0.222 0.138" rpy="0 3.1415 2.617901" />
             <geometry>
-                <mesh filename="file://$(find warehouse_robot_sim)/meshes/TriOrb300P100_Casters_BlockC_Pall.stl" scale="0.001 0.001 0.001" />
+                <mesh filename="file://$(find triorb_descriptions)/meshes/TriOrb300P100_Casters_BlockC_Pall.stl" scale="0.001 0.001 0.001" />
             </geometry>
         </collision>
@@ -330,5 +327,5 @@
             <origin xyz="0.057 0.222 0.138" rpy="0 3.1415 0.523599" />
             <geometry>
-                <mesh filename="file://$(find warehouse_robot_sim)/meshes/TriOrb300P100_Casters_BlockC_Pall.stl" scale="0.001 0.001 0.001" />
+                <mesh filename="file://$(find triorb_descriptions)/meshes/TriOrb300P100_Casters_BlockC_Pall.stl" scale="0.001 0.001 0.001" />
             </geometry>
             <material name="dark_gray">
@@ -339,5 +336,5 @@
             <origin xyz="0.057 0.222 0.138" rpy="0 3.1415 0.523599" />
             <geometry>
-                <mesh filename="file://$(find warehouse_robot_sim)/meshes/TriOrb300P100_Casters_BlockC_Pall.stl" scale="0.001 0.001 0.001" />
+                <mesh filename="file://$(find triorb_descriptions)/meshes/TriOrb300P100_Casters_BlockC_Pall.stl" scale="0.001 0.001 0.001" />
             </geometry>
         </collision>
@@ -352,5 +349,5 @@
             <origin xyz="0.221 -0.062 0.138" rpy="0 3.1415 0.521" />
             <geometry>
-                <mesh filename="file://$(find warehouse_robot_sim)/meshes/TriOrb300P100_Casters_BlockC_Pall.stl" scale="0.001 0.001 0.001" />
+                <mesh filename="file://$(find triorb_descriptions)/meshes/TriOrb300P100_Casters_BlockC_Pall.stl" scale="0.001 0.001 0.001" />
             </geometry>
             <material name="dark_gray">
@@ -361,5 +358,5 @@
             <origin xyz="0.221 -0.062 0.138" rpy="0 3.1415 0.521" />
             <geometry>
-                <mesh filename="file://$(find warehouse_robot_sim)/meshes/TriOrb300P100_Casters_BlockC_Pall.stl" scale="0.001 0.001 0.001" />
+                <mesh filename="file://$(find triorb_descriptions)/meshes/TriOrb300P100_Casters_BlockC_Pall.stl" scale="0.001 0.001 0.001" />
             </geometry>
         </collision>
@@ -374,5 +371,5 @@
             <origin xyz="0.164 -0.16 0.138" rpy="0 3.1415 -1.5734" />
             <geometry>
-                <mesh filename="file://$(find warehouse_robot_sim)/meshes/TriOrb300P100_Casters_BlockC_Pall.stl" scale="0.001 0.001 0.001" />
+                <mesh filename="file://$(find triorb_descriptions)/meshes/TriOrb300P100_Casters_BlockC_Pall.stl" scale="0.001 0.001 0.001" />
             </geometry>
             <material name="dark_gray">
@@ -383,5 +380,5 @@
             <origin xyz="0.164 -0.16 0.138" rpy="0 3.1415 -1.5734" />
             <geometry>
-                <mesh filename="file://$(find warehouse_robot_sim)/meshes/TriOrb300P100_Casters_BlockC_Pall.stl" scale="0.001 0.001 0.001" />
+                <mesh filename="file://$(find triorb_descriptions)/meshes/TriOrb300P100_Casters_BlockC_Pall.stl" scale="0.001 0.001 0.001" />
             </geometry>
         </collision>
@@ -396,5 +393,5 @@
             <origin xyz="-0.221 -0.062 0.138" rpy="0 3.1415 2.6154" />
             <geometry>
-                <mesh filename="file://$(find warehouse_robot_sim)/meshes/TriOrb300P100_Casters_BlockC_Pall.stl" scale="0.001 0.001 0.001" />
+                <mesh filename="file://$(find triorb_descriptions)/meshes/TriOrb300P100_Casters_BlockC_Pall.stl" scale="0.001 0.001 0.001" />
             </geometry>
             <material name="dark_gray">
@@ -405,5 +402,5 @@
             <origin xyz="-0.221 -0.062 0.138" rpy="0 3.1415 2.6154" />
             <geometry>
-                <mesh filename="file://$(find warehouse_robot_sim)/meshes/TriOrb300P100_Casters_BlockC_Pall.stl" scale="0.001 0.001 0.001" />
+                <mesh filename="file://$(find triorb_descriptions)/meshes/TriOrb300P100_Casters_BlockC_Pall.stl" scale="0.001 0.001 0.001" />
             </geometry>
         </collision>
@@ -418,5 +415,5 @@
             <origin xyz="-0.164 -0.16 0.138" rpy="0 3.1415 4.9715" />
             <geometry>
-                <mesh filename="file://$(find warehouse_robot_sim)/meshes/TriOrb300P100_Casters_BlockC_Pall.stl" scale="0.001 0.001 0.001" />
+                <mesh filename="file://$(find triorb_descriptions)/meshes/TriOrb300P100_Casters_BlockC_Pall.stl" scale="0.001 0.001 0.001" />
             </geometry>
             <material name="dark_gray">
@@ -427,5 +424,5 @@
             <origin xyz="-0.164 -0.16 0.138" rpy="0 3.1415 4.9715" />
             <geometry>
-                <mesh filename="file://$(find warehouse_robot_sim)/meshes/TriOrb300P100_Casters_BlockC_Pall.stl" scale="0.001 0.001 0.001" />
+                <mesh filename="file://$(find triorb_descriptions)/meshes/TriOrb300P100_Casters_BlockC_Pall.stl" scale="0.001 0.001 0.001" />
             </geometry>
         </collision>
@@ -470,5 +467,5 @@
             <origin xyz="-0.012 -0.133 0.07" rpy="0.0 0.0 -1.5708" />
             <geometry>
-                <mesh filename="file://$(find warehouse_robot_sim)/meshes/TriOrb300P100_PlateA_BLMR5100K-10-B_GPA28GT5150-A-N18.stl" scale="0.001 0.001 0.001" />
+                <mesh filename="file://$(find triorb_descriptions)/meshes/TriOrb300P100_PlateA_BLMR5100K-10-B_GPA28GT5150-A-N18.stl" scale="0.001 0.001 0.001" />
             </geometry>
             <material name="white_aluminum">
@@ -479,5 +476,5 @@
             <origin xyz="-0.012 -0.133 0.07" rpy="0.0 0.0 -1.5708" />
             <geometry>
-                <mesh filename="file://$(find warehouse_robot_sim)/meshes/TriOrb300P100_PlateA_BLMR5100K-10-B_GPA28GT5150-A-N18.stl" scale="0.001 0.001 0.001" />
+                <mesh filename="file://$(find triorb_descriptions)/meshes/TriOrb300P100_PlateA_BLMR5100K-10-B_GPA28GT5150-A-N18.stl" scale="0.001 0.001 0.001" />
             </geometry>
         </collision>
@@ -492,5 +489,5 @@
             <origin xyz="-0.012 -0.123 0.07" rpy="-1.5708 0.0 -1.5708" />
             <geometry>
-                <mesh filename="file://$(find warehouse_robot_sim)/meshes/TriOrb300P100_PlateA_BLMR5100K-10-B_Motor.stl" scale="0.001 0.001 0.001" />
+                <mesh filename="file://$(find triorb_descriptions)/meshes/TriOrb300P100_PlateA_BLMR5100K-10-B_Motor.stl" scale="0.001 0.001 0.001" />
             </geometry>
             <material name="light_gray">
@@ -501,5 +498,5 @@
             <origin xyz="-0.012 -0.123 0.07" rpy="-1.5708 0.0 -1.5708" />
             <geometry>
-                <mesh filename="file://$(find warehouse_robot_sim)/meshes/TriOrb300P100_PlateA_BLMR5100K-10-B_Motor.stl" scale="0.001 0.001 0.001" />
+                <mesh filename="file://$(find triorb_descriptions)/meshes/TriOrb300P100_PlateA_BLMR5100K-10-B_Motor.stl" scale="0.001 0.001 0.001" />
             </geometry>
         </collision>
@@ -514,5 +511,5 @@
             <origin xyz="0.123 0.057 0.067" rpy="0.0 0.0 0.523599" />
             <geometry>
-                <mesh filename="file://$(find warehouse_robot_sim)/meshes/TriOrb300P100_PlateA_BLMR5100K-10-B_GPA28GT5150-A-N18.stl" scale="0.001 0.001 0.001" />
+                <mesh filename="file://$(find triorb_descriptions)/meshes/TriOrb300P100_PlateA_BLMR5100K-10-B_GPA28GT5150-A-N18.stl" scale="0.001 0.001 0.001" />
             </geometry>
             <material name="white_aluminum">
@@ -523,5 +520,5 @@
             <origin xyz="0.123 0.057 0.067" rpy="0.0 0.0 0.523599" />
             <geometry>
-                <mesh filename="file://$(find warehouse_robot_sim)/meshes/TriOrb300P100_PlateA_BLMR5100K-10-B_GPA28GT5150-A-N18.stl" scale="0.001 0.001 0.001" />
+                <mesh filename="file://$(find triorb_descriptions)/meshes/TriOrb300P100_PlateA_BLMR5100K-10-B_GPA28GT5150-A-N18.stl" scale="0.001 0.001 0.001" />
             </geometry>
         </collision>
@@ -536,5 +533,5 @@
             <origin xyz="0.115 0.052 0.067" rpy="-1.5708 0.0 0.523599" />
             <geometry>
-                <mesh filename="file://$(find warehouse_robot_sim)/meshes/TriOrb300P100_PlateA_BLMR5100K-10-B_Motor.stl" scale="0.001 0.001 0.001" />
+                <mesh filename="file://$(find triorb_descriptions)/meshes/TriOrb300P100_PlateA_BLMR5100K-10-B_Motor.stl" scale="0.001 0.001 0.001" />
             </geometry>
             <material name="light_gray">
@@ -545,5 +542,5 @@
             <origin xyz="0.115 0.052 0.067" rpy="-1.5708 0.0 0.523599" />
             <geometry>
-                <mesh filename="file://$(find warehouse_robot_sim)/meshes/TriOrb300P100_PlateA_BLMR5100K-10-B_Motor.stl" scale="0.001 0.001 0.001" />
+                <mesh filename="file://$(find triorb_descriptions)/meshes/TriOrb300P100_PlateA_BLMR5100K-10-B_Motor.stl" scale="0.001 0.001 0.001" />
             </geometry>
         </collision>
@@ -558,5 +555,5 @@
             <origin xyz="-0.111 0.078 0.067" rpy="0.0 0.0 2.61799" />
             <geometry>
-                <mesh filename="file://$(find warehouse_robot_sim)/meshes/TriOrb300P100_PlateA_BLMR5100K-10-B_GPA28GT5150-A-N18.stl" scale="0.001 0.001 0.001" />
+                <mesh filename="file://$(find triorb_descriptions)/meshes/TriOrb300P100_PlateA_BLMR5100K-10-B_GPA28GT5150-A-N18.stl" scale="0.001 0.001 0.001" />
             </geometry>
             <material name="white_aluminum">
@@ -567,5 +564,5 @@
             <origin xyz="-0.111 0.078 0.067" rpy="0.0 0.0 2.61799" />
             <geometry>
-                <mesh filename="file://$(find warehouse_robot_sim)/meshes/TriOrb300P100_PlateA_BLMR5100K-10-B_GPA28GT5150-A-N18.stl" scale="0.001 0.001 0.001" />
+                <mesh filename="file://$(find triorb_descriptions)/meshes/TriOrb300P100_PlateA_BLMR5100K-10-B_GPA28GT5150-A-N18.stl" scale="0.001 0.001 0.001" />
             </geometry>
         </collision>
@@ -580,5 +577,5 @@
             <origin xyz="-0.103 0.073 0.067" rpy="-1.5708 0.0 2.61799" />
             <geometry>
-                <mesh filename="file://$(find warehouse_robot_sim)/meshes/TriOrb300P100_PlateA_BLMR5100K-10-B_Motor.stl" scale="0.001 0.001 0.001" />
+                <mesh filename="file://$(find triorb_descriptions)/meshes/TriOrb300P100_PlateA_BLMR5100K-10-B_Motor.stl" scale="0.001 0.001 0.001" />
             </geometry>
             <material name="light_gray">
@@ -589,5 +586,5 @@
             <origin xyz="-0.103 0.073 0.067" rpy="-1.5708 0.0 2.61799" />
             <geometry>
-                <mesh filename="file://$(find warehouse_robot_sim)/meshes/TriOrb300P100_PlateA_BLMR5100K-10-B_Motor.stl" scale="0.001 0.001 0.001" />
+                <mesh filename="file://$(find triorb_descriptions)/meshes/TriOrb300P100_PlateA_BLMR5100K-10-B_Motor.stl" scale="0.001 0.001 0.001" />
             </geometry>
         </collision>
@@ -632,5 +629,5 @@
             <origin xyz="0.0 -0.131 0.064" rpy="1.5708 0.0 0.0" />
             <geometry>
-                <mesh filename="file://$(find warehouse_robot_sim)/meshes/TriOrb300P100_PlateA_Belt.stl" scale="0.001 0.001 0.001" />
+                <mesh filename="file://$(find triorb_descriptions)/meshes/TriOrb300P100_PlateA_Belt.stl" scale="0.001 0.001 0.001" />
             </geometry>
             <material name="black">
@@ -641,5 +638,5 @@
             <origin xyz="0.0 -0.131 0.064" rpy="1.5708 0.0 0.0" />
             <geometry>
-                <mesh filename="file://$(find warehouse_robot_sim)/meshes/TriOrb300P100_PlateA_Belt.stl" scale="0.001 0.001 0.001" />
+                <mesh filename="file://$(find triorb_descriptions)/meshes/TriOrb300P100_PlateA_Belt.stl" scale="0.001 0.001 0.001" />
             </geometry>
         </collision>
@@ -654,5 +651,5 @@
             <origin xyz="0.115 0.067 0.061" rpy="1.5708 0.0 2.0944" />
             <geometry>
-                <mesh filename="file://$(find warehouse_robot_sim)/meshes/TriOrb300P100_PlateA_Belt.stl" scale="0.001 0.001 0.001" />
+                <mesh filename="file://$(find triorb_descriptions)/meshes/TriOrb300P100_PlateA_Belt.stl" scale="0.001 0.001 0.001" />
             </geometry>
             <material name="black">
@@ -663,5 +660,5 @@
             <origin xyz="0.115 0.067 0.061" rpy="1.5708 0.0 2.0944" />
             <geometry>
-                <mesh filename="file://$(find warehouse_robot_sim)/meshes/TriOrb300P100_PlateA_Belt.stl" scale="0.001 0.001 0.001" />
+                <mesh filename="file://$(find triorb_descriptions)/meshes/TriOrb300P100_PlateA_Belt.stl" scale="0.001 0.001 0.001" />
             </geometry>
         </collision>
@@ -676,5 +673,5 @@
             <origin xyz="-0.115 0.067 0.061" rpy="1.5708 0.0 -2.0944" />
             <geometry>
-                <mesh filename="file://$(find warehouse_robot_sim)/meshes/TriOrb300P100_PlateA_Belt.stl" scale="0.001 0.001 0.001" />
+                <mesh filename="file://$(find triorb_descriptions)/meshes/TriOrb300P100_PlateA_Belt.stl" scale="0.001 0.001 0.001" />
             </geometry>
             <material name="black">
@@ -685,5 +682,5 @@
             <origin xyz="-0.115 0.067 0.061" rpy="1.5708 0.0 -2.0944" />
             <geometry>
-                <mesh filename="file://$(find warehouse_robot_sim)/meshes/TriOrb300P100_PlateA_Belt.stl" scale="0.001 0.001 0.001" />
+                <mesh filename="file://$(find triorb_descriptions)/meshes/TriOrb300P100_PlateA_Belt.stl" scale="0.001 0.001 0.001" />
             </geometry>
         </collision>
@@ -713,5 +710,5 @@
             <origin xyz="-0.094 -0.153 0.084" rpy="0.0 0.0 1.5708" />
             <geometry>
-                <mesh filename="file://$(find warehouse_robot_sim)/meshes/TriOrb300P100_PlateA_Axis_GPA25GT5150-A-N15.stl" scale="0.001 0.001 0.001" />
+                <mesh filename="file://$(find triorb_descriptions)/meshes/TriOrb300P100_PlateA_Axis_GPA25GT5150-A-N15.stl" scale="0.001 0.001 0.001" />
             </geometry>
             <material name="white_aluminum">
@@ -722,5 +719,5 @@
             <origin xyz="-0.094 -0.153 0.084" rpy="0.0 0.0 1.5708" />
             <geometry>
-                <mesh filename="file://$(find warehouse_robot_sim)/meshes/TriOrb300P100_PlateA_Axis_GPA25GT5150-A-N15.stl" scale="0.001 0.001 0.001" />
+                <mesh filename="file://$(find triorb_descriptions)/meshes/TriOrb300P100_PlateA_Axis_GPA25GT5150-A-N15.stl" scale="0.001 0.001 0.001" />
             </geometry>
         </collision>
@@ -735,5 +732,5 @@
             <origin xyz="0.094 -0.153 0.084" rpy="0.0 0.0 1.5708" />
             <geometry>
-                <mesh filename="file://$(find warehouse_robot_sim)/meshes/TriOrb300P100_PlateA_Axis_GPA25GT5150-A-N15.stl" scale="0.001 0.001 0.001" />
+                <mesh filename="file://$(find triorb_descriptions)/meshes/TriOrb300P100_PlateA_Axis_GPA25GT5150-A-N15.stl" scale="0.001 0.001 0.001" />
             </geometry>
             <material name="white_aluminum">
@@ -744,5 +741,5 @@
             <origin xyz="0.094 -0.153 0.084" rpy="0.0 0.0 1.5708" />
             <geometry>
-                <mesh filename="file://$(find warehouse_robot_sim)/meshes/TriOrb300P100_PlateA_Axis_GPA25GT5150-A-N15.stl" scale="0.001 0.001 0.001" />
+                <mesh filename="file://$(find triorb_descriptions)/meshes/TriOrb300P100_PlateA_Axis_GPA25GT5150-A-N15.stl" scale="0.001 0.001 0.001" />
             </geometry>
         </collision>
@@ -757,5 +754,5 @@
             <origin xyz="-0.087 0.159 0.081" rpy="0.0 0.0 -0.523599" />
             <geometry>
-                <mesh filename="file://$(find warehouse_robot_sim)/meshes/TriOrb300P100_PlateA_Axis_GPA25GT5150-A-N15.stl" scale="0.001 0.001 0.001" />
+                <mesh filename="file://$(find triorb_descriptions)/meshes/TriOrb300P100_PlateA_Axis_GPA25GT5150-A-N15.stl" scale="0.001 0.001 0.001" />
             </geometry>
             <material name="white_aluminum">
@@ -766,5 +763,5 @@
             <origin xyz="-0.087 0.159 0.081" rpy="0.0 0.0 -0.523599" />
             <geometry>
-                <mesh filename="file://$(find warehouse_robot_sim)/meshes/TriOrb300P100_PlateA_Axis_GPA25GT5150-A-N15.stl" scale="0.001 0.001 0.001" />
+                <mesh filename="file://$(find triorb_descriptions)/meshes/TriOrb300P100_PlateA_Axis_GPA25GT5150-A-N15.stl" scale="0.001 0.001 0.001" />
             </geometry>
         </collision>
@@ -779,5 +776,5 @@
             <origin xyz="-0.181 -0.004 0.081" rpy="0.0 0.0 -0.523599" />
             <geometry>
-                <mesh filename="file://$(find warehouse_robot_sim)/meshes/TriOrb300P100_PlateA_Axis_GPA25GT5150-A-N15.stl" scale="0.001 0.001 0.001" />
+                <mesh filename="file://$(find triorb_descriptions)/meshes/TriOrb300P100_PlateA_Axis_GPA25GT5150-A-N15.stl" scale="0.001 0.001 0.001" />
             </geometry>
             <material name="white_aluminum">
@@ -788,5 +785,5 @@
             <origin xyz="-0.181 -0.004 0.081" rpy="0.0 0.0 -0.523599" />
             <geometry>
-                <mesh filename="file://$(find warehouse_robot_sim)/meshes/TriOrb300P100_PlateA_Axis_GPA25GT5150-A-N15.stl" scale="0.001 0.001 0.001" />
+                <mesh filename="file://$(find triorb_descriptions)/meshes/TriOrb300P100_PlateA_Axis_GPA25GT5150-A-N15.stl" scale="0.001 0.001 0.001" />
             </geometry>
         </collision>
@@ -801,5 +798,5 @@
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